File: audio-simple-se/simple-se.sch (EAGLE design)
At the start: 57 parts, among them IC3 10M45, IC4 10M45, J1 6.3VAC, X10 C_FILTER, X11 L_IN, X12 R_IN, X13 6.3VAC, X2 5VAC, X3 CFB_R, X4 CFB_L, X5 L_FILTER, X8 750VAC, X9 CON_B+

Commit message: Added M3 PEM nuts to library
Parts:
- added X1, X14: PEM-SMTSO-M3, simple-se:PEM-SMTSO-M3
Connections:
- net GND: now also X1.P$1, X14.P$1
Other:
- note added: "10mA CCS"
- note added: "Dist: D.B. Roberts Company"

Commit message: Added SPOX Connectors, Added Heater Linear Supply
Parts:
- removed J3: (no value), con-amp:MTA02-156
- removed J4: (no value), con-amp:MTA03-156
- removed X11: L_IN, con-ptr500:AK500/2
- removed X12: R_IN, con-ptr500:AK500/2
- added C13: 56u, rcl:CPOL-EUE10-22.5
- added C14: 15m, rcl:CPOL-EUE7.5-18
- added C15, C16: 100n, rcl:C-EU050-055X075
- added C6: 470n, 100V, rcl:C-EU075-063X106
- added IC1: LT4320, simple-se:LT4320
- added IC2: MIC29502WT, Kramnik's Library:MIC29502WT
- added KK4: SK129-PAD, heatsink:SK129-PAD
- added R20: 100R, 1%, rcl:R-EU_0207/12
- added R24: 412R, 1%, rcl:R-EU_0207/12
- added S1, S2, S3, S4: (no value), sc_usercreated:MOSFET-N_DPAK
- added X15: PSU-HV, simple-se:MOLEX-SPOX-5281-3POS
- added X16: OPT-PRI-R, simple-se:MOLEX-SPOX-5281-3POS
- C10: value 0.47uF 100V -> 120u; device rcl:C-US075-063X106 -> rcl:CPOL-EUE10-30
- C8: value 120uF -> 15m; device rcl:CPOL-USE10-30 -> rcl:CPOL-EUE7.5-18
- C9: value 56uF -> 15m; device rcl:CPOL-USE10-22.5 -> rcl:CPOL-EUE7.5-18
- J1: value 6.3VAC -> IN-R
- J2: value (none) -> IN-L
- V7: value (none) -> 5AR4
- X10: device con-ptr500:AK500/3 -> simple-se:MOLEX-SPOX-5281-2POS; OC_FARNELL unknown -> (none); OC_NEWARK unknown -> (none)
- X13: value 6.3VAC -> L_FILTER; device con-ptr500:AK500/3 -> simple-se:MOLEX-SPOX-5281-2POS; OC_FARNELL unknown -> (none); OC_NEWARK unknown -> (none)
- X2: value 5VAC -> OPT-PRI-L; device con-ptr500:AK500/2 -> simple-se:MOLEX-SPOX-5281-3POS; OC_FARNELL unknown -> (none); OC_NEWARK unknown -> (none)
- X3: value CFB_R -> PSU-STANDBY; device con-ptr500:AK500/2 -> simple-se:MOLEX-SPOX-5281-2POS; OC_FARNELL unknown -> (none); OC_NEWARK unknown -> (none)
- X4: value CFB_L -> TRIODE-UL-SW-R; device con-ptr500:AK500/2 -> simple-se:MOLEX-SPOX-5281-3POS; OC_FARNELL unknown -> (none); OC_NEWARK unknown -> (none)
- X5: value L_FILTER -> TRIODE-UL-SW-L; device con-ptr500:AK500/2 -> simple-se:MOLEX-SPOX-5281-3POS; OC_FARNELL unknown -> (none); OC_NEWARK unknown -> (none)
- X6: value (none) -> CFB-L; device con-ptr500:AK500/3 -> simple-se:MOLEX-SPOX-5281-2POS
- X7: value (none) -> CFB-R; device con-ptr500:AK500/3 -> simple-se:MOLEX-SPOX-5281-2POS
- X8: value 750VAC -> PSU-5VAC; device con-ptr500:AK500/3 -> simple-se:MOLEX-SPOX-5281-2POS; OC_FARNELL unknown -> (none); OC_NEWARK unknown -> (none)
- X9: value CON_B+ -> PSU-6V3AC; device con-ptr500:AK500/2 -> simple-se:MOLEX-SPOX-5281-3POS; OC_FARNELL unknown -> (none); OC_NEWARK unknown -> (none)
Connections:
- removed net N$23 (its old number): R23.1, X7-2.KL
- removed net N$38: V1".H2, V5".H2, V6".H2, X13-1.KL
- new net N$29: R23.1, X4.2
- new net N$42: IC1.BG2, S4.G
- new net N$43: IC1.TG2, S2.G
- new net N$44: IC1.IN2, S2.S, S3.D, X9.1
- new net N$45: IC1.BG1, S3.G
- new net N$46: C14.-, C15.2, C16.2, C8.-, C9.-, IC1.OUTN, IC2.GND, R20.1, S3.S, S4.S, V1".H2, V5".H2, V6".H2
- new net N$47: C14.+, C16.1, C6.1, IC2.OUT, R16.2, R21.1, R24.1, V1".H1, V1".H3, V5".H1, V6".H1
- new net N$49: IC2.SENSE, R20.2, R24.2
- new net NC_6V3AC_CT: X9.2
- new net OPT-MINUS-L: V5G$1.PA, X2.2, X5.1
- new net OPT-UL-TAP-L: X2.3, X5.3
- net B+: now also C10.+, X10.1, X13.2, X16.1, X2.1; no longer C8.+, X10-3.KL, X5-1.KL, X9-1.KL, X9-2.KL
- net GND: now also C10.-, C13.-, C6.2, J1.2, J2.2, X10.2, X3.2, X6.2, X7.2; no longer C10.2, C8.-, C9.-, X10-1.KL, X10-2.KL, X11-2.KL, X12-1.KL, X3-1.KL, X4-2.KL, X8-2.KL
- net LOUT_PLATE: now also X16.2, X4.1; no longer X7-3.KL
- net LOUT_SCREEN: now also X16.3, X4.3; no longer X7-1.KL
- net N$10: now also J2.1; no longer X12-2.KL
- net N$19: now also X6.1; no longer X3-2.KL
- net N$21: now also X5.2; no longer X6-2.KL
- net N$22: now also X15.2, X3.1; no longer V5G$1.PA, X6-1.KL
- net N$25: now also C13.+, X13.1, X8.2; no longer C9.+, X2-1.KL, X5-2.KL
- net N$26: now also X15.1; no longer X8-1.KL
- net N$27: now also IC1.TG1, S1.G; no longer V1".H1, V1".H3, V5".H1, V6".H1, X13-3.KL
- net N$33: now also X15.3; no longer X8-3.KL
- net N$34: now also IC1.IN1, S1.S, S4.D, X9.3; no longer X6-3.KL
- net N$35: now also X8.1; no longer X2-2.KL
- net N$40: now also X7.1; no longer X4-1.KL
- net N$41: now also C15.1, C8.+, C9.+, IC1.OUTP, IC2.!SHDN, IC2.IN, S1.D, S2.D; no longer C10.1, R16.2, R21.1, X13-2.KL
- net N$9: now also J1.1; no longer X11-1.KL
Other:
- note added: "! Do Not Tie to Chassis GND"
- note added: "0.3A"
- note added: "1.6A"
- note added: "5.0A Adj. Linear Regulator"
- note added: "Design for Vout = 6.3V"
- note added: "I_heater ="
- note added: "LEFT CHANNEL"
- note added: "RIGHT CHANNEL"
- note added: "Ra"
- note added: "Rb"
- note added: "Vout = 1.240 * (Ra/Rb + 1)"
- moved on the sheet: C3, C4, C8, C9, J1, J2, R16, R17, R19, R21, R22, R23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

Commit message: Added Quench Circuit Directory
Parts:
- added B1: RECTIFIER-GBU4, rectifier:RECTIFIER-GBU4
- added C17: 100n, rcl:C-EU102-043X133
- added C18: 1500u, 63V, rcl:CPOL-EUE5-13
- added C19, C20: 100n, 630V, rcl:C-EU150-072X183
- added C21: 100n, rcl:C-EU150-072X183
- added C22: 10u, 630V, rcl:C-EU150-072X183
- added D10: 1N5342, diode:ZENER-DIODEDO35Z10
- added D8, D9: 1N4007, diode:1N4004
- added IC5, IC6: 10M45, simple-se:10M45V
- added IC9: LM317, v-reg:LM317TS
- added J4: STAGE1-SEL-L, con-amp:MTA03-156
- added J5: STAGE1-SEL-R, con-amp:MTA03-156
- added KK3: SK129-PAD, heatsink:SK129-PAD
- added R25: 10R, 3W, rcl:R-EU_0617/17
- added R26: 191R, rcl:R-EU_0309/12
- added R27: R_FILTER, rcl:R-EU_0922/22
- added R28: 1R, rcl:R-EU_0309/12
- added R29, R31: 1k, rcl:R-EU_0309/12
- added R30: 1k, pot:TRIM_EU-S64W
- added R32: 68.1k, rcl:R-EU_0309/12
- added R34, R35: 10R, rcl:R-EU_0309/12
- added R36: 6k2, rcl:R-EU_0309/12
- added T3: BUL416T, transistor:-NPN-TO220V
- added X11: PEM-SMTSO-M3, simple-se:PEM-SMTSO-M3
- added X12: OPT-SEC-L, simple-se:MOLEX-SPOX-5281-2POS
- added X17: SPKR-L, simple-se:MOLEX-SPOX-5281-2POS
- added X18: SPKR-R, simple-se:MOLEX-SPOX-5281-2POS
- added X19: CFB-SW-R, simple-se:MOLEX-SPOX-5281-3POS
- C1: value 1500u 63V -> 1500u, 6.3V; device rcl:CPOL-USE5-10.5 -> rcl:CPOL-EUE5-10.5
- C11, C7: value 0.1uF 400V -> 100n, 630V; device rcl:C-US102-064X133 -> rcl:C-EU150-072X183
- C12, C5: device rcl:C-EU225-113X268 -> rcl:C-EU275-113X316
- C14: value 15m -> 15m, 10V
- C2: value 1500u 6.3V -> 1500u, 6.3V; device rcl:CPOL-USE5-10.5 -> rcl:CPOL-EUE5-10.5
- C3: value 1500u 63V -> 1500u, 63V; device rcl:CPOL-USE5-13 -> rcl:CPOL-EUE5-13
- C4: value 1500u 63V -> 100n, 630V; device rcl:CPOL-USE5-13 -> rcl:C-EU150-072X183
- C8, C9: value 15m -> 15m, 16V
- R1, R10, R11, R12, R13, R15, R2, R20, R24, R3, R4, R5, R6, R7, R8, R9: device rcl:R-EU_0207/12 -> rcl:R-EU_0309/12
- X15: value PSU-HV -> PSU-HV-IN
- X3: value PSU-STANDBY -> PSU-STANDBY-SW
- X6: value CFB-L -> CFB-SW-L; device simple-se:MOLEX-SPOX-5281-2POS -> simple-se:MOLEX-SPOX-5281-3POS
- X7: value CFB-R -> OPT-SEC-R
- X8: value PSU-5VAC -> PSU-5VAC-IN
- X9: value PSU-6V3AC -> PSU-6V3AC-IN
Connections:
- net LOUT_PLATE renamed OPT-MINUS-R
- net LOUT_SCREEN renamed OPT-UL-TAP-R
- net N$12 renamed SCREEN-GRID-L
- net N$21 renamed SCREEN-GRID-CONN-L
- net N$23 renamed SCREEN-GRID-R
- net N$29 renamed SCREEN-GRID-CONN-R
- new net HV_LFILT: C10.+, D9.C, R27.1, R35.2, R36.2, X10.1, X13.2
- new net HV_RECT: C13.+, R27.2, V7.H1, X13.1, X8.2
- new net N$12: B1.+, B1.-
- new net N$21: B1.AC1, C17.1, R25.2, X11.P$1
- new net N$23: X12.1, X17.1, X6.1
- new net N$24: R35.1, T3.C
- new net N$28: C21.1, R34.2, T3.E
- new net N$29: C20.1, C21.2, IC9.IN, R34.1
- new net N$36: X19.2
- new net N$37: X18.1, X19.1, X7.1
- new net N$38: C22.1, R28.1
- new net N$48: D10.C, R36.1, T3.B
- new net N$50: IC5.G, R29.2
- new net N$51: IC5.A, R14.2
- new net N$52: C12.2, J4.2
- new net N$53: IC4.A, IC6.K
- new net N$54: IC6.G, R31.2
- new net N$55: C5.1, J5.2
- net B+: now also C19.1, D10.A, D8.C, D9.A, IC9.OUT, R26.2, R30.E; no longer C10.+, X10.1, X13.2
- net GND: now also B1.AC2, C17.2, C19.2, C20.2, C22.2, C4.2, R25.1, R32.1, X12.2, X17.2, X18.2, X19.3, X6.3; no longer X6.2
- net N$14: now also C12.1; no longer C12.2
- net N$15: now also C1.+; no longer C2.+
- net N$16: now also C2.+; no longer C1.+
- net N$17: now also IC6.A; no longer IC4.A
- net N$18: now also IC5.K; no longer R14.2
- net N$19: now also C18.-, X6.2; no longer C3.-, X6.1
- net N$2: now also J4.3; no longer C12.1
- net N$25: now also C4.1, D8.A, IC9.ADJ, R26.1, R28.2, R30.A, R30.S, R32.2; no longer C13.+, V7.H1, X13.1, X8.2
- net N$30: now also C11.2, C18.+; no longer C3.+, C7.2
- net N$31: now also C7.1; no longer C11.1
- net N$32: now also C3.+, C7.2; no longer C11.2, C4.+
- net N$39: now also C11.1; no longer C7.1
- net N$4: now also J5.3; no longer C5.1
- net N$40: now also C3.-; no longer C4.-, X7.1
- net N$5: now also J5.1, R31.1
- net N$7: now also J4.1, R29.1
Other:
- note added: ""Hazen Grid Mod""
- note added: "283-10-RC"
- note added: "6.8V Zener"
- note added: "This cap. is weird, read:"
- note added: "Tie to Chassis GND Here"
- note added: "http://www.decware.com/newsite/paper145.htm"
- moved on the sheet: C1, C10, C11, C12, C13, C14, C15, C16, C2, C3, C5, C6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
