File: 6301-tutorial/tut1.sch (EAGLE design)
At the start: 14 parts, among them Q1 2N3904, Q2 2N3904

Commit message: Added layout
Parts:
- added H1: MOUNT-PAD-ROUND3.2, holes:MOUNT-PAD-ROUND3.2
- JP1: value (none) -> VIN
- JP2: value (none) -> VOUT
- JP3: value (none) -> POWER
- R5: value (none) -> 10k
Connections:
- net N$5 renamed VO
- net GND: now also H1.MOUNT
Changed lines of the file:
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@@
 </variantdefs>
 <classes>
-<class number="0" name="default" width="0" drill="0">
+<class number="0" name="default" width="0.8128" drill="0">
 </class>
 </classes>
@@
 <part name="R3" library="rcl" deviceset="R-EU_" device="0207/10" value="1M"/>
 <part name="R4" library="rcl" deviceset="R-EU_" device="0207/10" value="1M"/>
-<part name="R5" library="rcl" deviceset="R-EU_" device="0207/10"/>
+<part name="R5" library="rcl" deviceset="R-EU_" device="0207/10" value="10k"/>
 <part name="R6" library="rcl" deviceset="R-EU_" device="0207/10" value="1k"/>
 <part name="C1" library="rcl" deviceset="CPOL-EU" device="E5-10.5" value="100u"/>
 <part name="C2" library="rcl" deviceset="C-EU" device="050-025X075" value="100n"/>
 <part name="C3" library="rcl" deviceset="C-EU" device="050-025X075" value="100n"/>
-<part name="JP1" library="jumper" deviceset="JP1E" device=""/>
-<part name="JP2" library="jumper" deviceset="JP1E" device=""/>
+<part name="JP1" library="jumper" deviceset="JP1E" device="" value="VIN"/>
+<part name="JP2" library="jumper" deviceset="JP1E" device="" value="VOUT"/>
 <part name="GND1" library="supply1" deviceset="GND" device=""/>
 <part name="GND2" library="supply1" deviceset="GND" device=""/>
@@
 <part name="GND4" library="supply1" deviceset="GND" device=""/>
 <part name="GND5" library="supply1" deviceset="GND" device=""/>
-<part name="JP3" library="jumper" deviceset="JP1E" device=""/>
+<part name="JP3" library="jumper" deviceset="JP1E" device="" value="POWER"/>
 <part name="GND6" library="supply1" deviceset="GND" device=""/>
 <part name="FRAME1" library="frames" deviceset="FRAME_A_L" device=""/>
+<part name="H1" library="holes" deviceset="MOUNT-PAD-ROUND" device="3.2"/>
+<part name="GND7" library="supply1" deviceset="GND" device=""/>
 </parts>
 <sheets>
@@
 <instance part="FRAME1" gate="G$1" x="0" y="0"/>
 <instance part="FRAME1" gate="G$2" x="172.72" y="0"/>
+<instance part="H1" gate="G$1" x="175.26" y="144.78"/>
+<instance part="GND7" gate="1" x="170.18" y="139.7"/>
 </instances>
 <busses>
@@
 </segment>
 </net>
-<net name="N$5" class="0">
+<net name="VO" class="0">
 <segment>
 <pinref part="R5" gate="G$1" pin="1"/>
@@
 <pinref part="C3" gate="G$1" pin="1"/>
 <junction x="119.38" y="119.38"/>
+<label x="121.92" y="121.92" size="1.778" layer="95"/>
 </segment>
 </net>
@@
 <wire x1="170.18" y1="91.44" x2="172.72" y2="91.44" width="0.1524" layer="91"/>
 </segment>
-</net>
+<segment>
+<pinref part="H1" gate="G$1" pin="MOUNT"/>
+<wire x1="172.72" y1="144.78" x2="170.18" y2="144.78" width="0.1524" layer="91"/>
+<pinref part="GND7" gate="1" pin="GND"/>
+<wire x1="170.18" y1="144.78" x2="170.18" y2="142.24" width="0.1524" layer="91"/>
+</segment>
+</net>
