File: audio-simple-differential-electrostatic/simple-differential-power-supply-rev1.brd (EAGLE design)
At the start: 160 x 100 mm, 22 parts, among them IC1 10M45, Q4 STF2N80K5, T1 BC559, T2 BC560

Commit message: t
Parts:
- added C10, C11, C12, C13: 1n, rcl:C225-087X268
- added C14: (no value), rcl:EB25D
- added C8: 100n, rcl:C050-025X075
- added C9: 10u, 500V, rcl:EB25D
- added D10, D11, D13, D9: MBR735, diode:TO220ACS
- added D7, D8: 1N4004, diode:DO41-10
- added IC2: 10M45, Kramnik's Library:TO220V
- added J2: VOUT_PLATE, Kramnik's Library:CONN_MOLEX_3PIN_MINI-FIT_JR
- added KK1, KK4, KK5: SK104-PAD, heatsink:SK104-PAD
- added KK2, KK3: SK129-PAD, heatsink:SK129
- added Q1: STF2N80K5, Kramnik's Library:TO220BV
- added R10: 110R, rcl:0309/10
- added R6: 4k7, rcl:0309/10
- added R7, R8: 225k, rcl:0309/10
- added R9: 15k, rcl:0309/10
- added T3: BC559, transistor-neu-to92:TO92-EBC
- added T4: BC560, transistor-neu-to92:TO92-EBC
- added X2: VOUT_OPAMP, con-molex:KK-156-3
- added X4: VOUT_HEATER, con-molex:KK-156-2
- moved IC1 145.3 mm to (-82.5, -74.9)
Connections:
- net N$1 renamed SREG_CASC_MID_L
- net N$2 renamed SREG_DIVIDER_L_BUF
- net N$5 renamed SREG_DIVIDER_L
- new net N$1: C11.2, C13.1, D10.C, D9.A
- new net N$10: KK5.K2
- new net N$13: KK3.A2,5
- new net N$14: KK3.B2,5
- new net N$16: KK1.K2
- new net N$17: X2.3
- new net N$18: X2.1
- new net N$19: X4.2
- new net N$2: C10.2, C12.1, D11.C, D13.A
- new net N$20: X4.1
- new net N$3: KK4.K1
- new net N$5: KK4.K2
- new net N$6: KK2.A2,5
- new net N$7: R7.1, R8.2
- new net N$8: KK2.B2,5
- new net PP_P450V_RIGHT: C9.+, IC1.1, J2.3, Q1.D, R10.1, R7.2
- new net PP_PFILAMENT_UNREG: C10.1, C11.1, C14.+, D13.C, D9.C
- new net SREG_CASC_MID_R: Q1.S, T3.C
- new net SREG_CCS_BIAS_L: IC2.3, R1.2
- new net SREG_CCS_BIAS_R: IC1.3, R10.2
- new net SREG_DIVIDER_R: C9.-, D7.C, D8.A, R8.1, R9.2, T4.B
- new net SREG_DIVIDER_R_BUF: R6.1, T3.B, T4.E
- net GND: now also C12.2, C13.2, C14.-, C8.2, D10.A, D11.A, D7.A, D8.C, J2.2, T3.E, X2.2
- net N$9: now also KK5.K1; no longer IC1.3, R1.2
- net PP_N15V0_ANALOG: now also R9.1, T4.C
- net PP_P15V0_ANALOG: now also C8.1, Q1.G, R6.2
- net PP_P450V_LEFT: now also IC2.1, J2.1; no longer IC1.1
- net PP_PB+_UNREG: now also IC2.2
