File: audio-simple-differential-electrostatic/simple-differential-power-supply-rev1.sch (EAGLE design)
At the start: 22 parts, among them IC1 10M45, Q4 STF2N80K5, T1 BC559, T2 BC560

Commit message: t
Parts:
- added C10, C11, C12, C13: 1n, rcl:C-EU225-087X268
- added C14: (no value), rcl:CPOL-EUE10-25
- added C8: 100n, rcl:C-EU050-025X075
- added C9: 10u, 500V, rcl:CPOL-EUE10-25
- added D10, D11, D13, D9: MBR735, diode:DIODE-TO220V
- added D7, D8: 1N4004, diode:1N4004
- added IC2: 10M45, Kramnik's Library:10M45V
- added J2: VOUT_PLATE, Kramnik's Library:CONN_MOLEX_3PIN_MINI-FIT_JR
- added KK1, KK4, KK5: SK104-PAD, heatsink:SK104-PAD
- added KK2, KK3: SK129-PAD, heatsink:SK129-PAD
- added Q1: STF2N80K5, Kramnik's Library:IRF540
- added R10: 110R, rcl:R-EU_0309/10
- added R6: 4k7, rcl:R-EU_0309/10
- added R7, R8: 225k, rcl:R-EU_0309/10
- added R9: 15k, rcl:R-EU_0309/10
- added T3: BC559, transistor-neu-to92:2N5088-NPN-TO92-EBC
- added T4: BC560, transistor-neu-to92:2N5087-PNP-TO92-EBC
- added X2: VOUT_OPAMP, con-molex:KK-156-3
- added X4: VOUT_HEATER, con-molex:KK-156-2
Connections:
- net N$1 renamed SREG_CASC_MID_L
- net N$2 renamed SREG_DIVIDER_L_BUF
- net N$5 renamed SREG_DIVIDER_L
- new net N$1: C11.2, C13.1, D10.C, D9.A
- new net N$10: KK5.K@2
- new net N$13: KK3.K@1
- new net N$14: KK3.K@2
- new net N$16: KK1.K@2
- new net N$17: X2-3.S
- new net N$18: X2-1.S
- new net N$19: X4-2.S
- new net N$2: C10.2, C12.1, D11.C, D13.A
- new net N$20: X4-1.S
- new net N$3: KK4.K@1
- new net N$5: KK4.K@2
- new net N$6: KK2.K@1
- new net N$7: R7.1, R8.2
- new net N$8: KK2.K@2
- new net PP_P450V_RIGHT: C9.+, IC1.G, J2.3, Q1.D, R10.1, R7.2
- new net PP_PFILAMENT_UNREG: C10.1, C11.1, C14.+, D13.C, D9.C
- new net SREG_CASC_MID_R: Q1.S, T3.C
- new net SREG_CCS_BIAS_L: IC2.K, R1.2
- new net SREG_CCS_BIAS_R: IC1.K, R10.2
- new net SREG_DIVIDER_R: C9.-, D7.C, D8.A, R8.1, R9.2, T4.B
- new net SREG_DIVIDER_R_BUF: R6.1, T3.B, T4.E
- net GND: now also C12.2, C13.2, C14.-, C8.2, D10.A, D11.A, D7.A, D8.C, J2.2, T3.E, X2-2.S
- net N$9: now also KK5.K@1; no longer IC1.K, R1.2
- net PP_N15V0_ANALOG: now also R9.1, T4.C
- net PP_P15V0_ANALOG: now also C8.1, Q1.G, R6.2
- net PP_P450V_LEFT: now also IC2.G, J2.1; no longer IC1.G
- net PP_PB+_UNREG: now also IC2.A
Other:
- note added: "1"
- note added: "1.0"
- note added: "15V"
- note added: "2"
- note added: "2 of 2"
- note added: "3"
- note added: "380V (71mA), 6.3V (2.5A)"
- note added: "450V"
- note added: "CONTENTS"
- note added: "Daniel Kramnik"
- note added: "Digikey HM1572-ND"
- note added: "Hammond 269EX"
- note added: "Keep appropriate clearances to high_voltage net class"
- note added: "MBR735GOS-ND"
- note added: "Net Class: high_voltage"
- note added: "Note: Shunt reg. is tolerant of CCS thermal variations, so cascode is not necessary"
- note added: "Power Transformer:"
- note added: "RECTIFICATION"
- note added: "Routing Notes:"
- note added: "SHEET"
- note added: "SHUNT REGULATORS"
- note added: "SIMPLE DIFFERENTIAL ELECTROSTATIC PSU BOARD"
- note added: "TABLE OF CONTENTS"
- note added: "https://www.hammfg.com/electronics/transformers/classic/200.pdf"
- note removed: "Note: Shunt reg. is tolerant of CCS thermal variations, so there is little advantage to a cascode"
