File: meng-spad-quenching/wire-bonding/cryobondr-qbit2.brd (EAGLE design)
At the start: 40 x 36 mm, 4 parts

Commit message: Work on cryobondr1 PCB
Parts:
- added IC1: QBIT2-WIREBOND-CRYO1, meng:QBIT2-WIREBOND-CRYO1
- added X1: CONN-D3, meng:MMCX-SMT
- added X2: CONN-D5, meng:MMCX-SMT
- added X3: CONN-D4, meng:MMCX-SMT
- added X4: CONN-D2, meng:MMCX-SMT
- added X5: CONN-D1, meng:MMCX-SMT
- added X6: CONN-D6, meng:MMCX-SMT
- added X7: CONN-D7, meng:MMCX-SMT
- added X8: CONN-D8, meng:MMCX-SMT
Connections:
- new net D1-N-CATHODE: IC1.D1-N-CATHODE, X5.S
- new net D1-P-ANODE: IC1.D1-P-ANODE, X5.G1, X5.G2, X5.G3, X5.G4
- new net D2-N-CATHODE: IC1.D2-N-CATHODE, X4.S
- new net D2-P-ANODE: IC1.D2-P-ANODE, X4.G1, X4.G2, X4.G3, X4.G4
- new net D3-N-CATHODE: IC1.D3-N-CATHODE, X1.S
- new net D3-P-ANODE: IC1.D3-P-ANODE, X1.G1, X1.G2, X1.G3, X1.G4
- new net D4-N-CATHODE: IC1.D4-N-CATHODE, X3.S
- new net D4-P-ANODE: IC1.D4-P-ANODE, X3.G1, X3.G2, X3.G3, X3.G4
- new net D5-N-CATHODE: IC1.D5-N-CATHODE, X2.S
- new net D5-P-ANODE: IC1.D5-P-ANODE, X2.G1, X2.G2, X2.G3, X2.G4
- new net D6-N-CATHODE: IC1.D6-N-CATHODE, X6.S
- new net D6-P-ANODE: IC1.D6-P-ANODE, X6.G1, X6.G2, X6.G3, X6.G4
- new net D7-N-CATHODE: IC1.D7-N-CATHODE, X7.S
- new net D7-P-ANODE: IC1.D7-P-ANODE, X7.G1, X7.G2, X7.G3, X7.G4
- new net D8-N-CATHODE: IC1.D8-N-CATHODE, X8.S
- new net D8-P-ANODE: IC1.D8-P-ANODE, X8.G1, X8.G2, X8.G3, X8.G4
Routing:
- net D1-P-ANODE: track 0.00 -> 23.2 mm
- net D3-P-ANODE: track 0.00 -> 22.3 mm
- net D8-P-ANODE: track 0.00 -> 21.2 mm
- net D2-P-ANODE: track 0.00 -> 18.6 mm
- net D6-P-ANODE: track 0.00 -> 18.3 mm
- net D5-P-ANODE: track 0.00 -> 17.7 mm
- net D1-N-CATHODE: track 0.00 -> 16.8 mm
- net D7-P-ANODE: track 0.00 -> 16.6 mm
- net D3-N-CATHODE: track 0.00 -> 16.2 mm
- net D4-P-ANODE: track 0.00 -> 15.8 mm
- net D8-N-CATHODE: track 0.00 -> 14.1 mm
- net D2-N-CATHODE: track 0.00 -> 13.0 mm
- net D5-N-CATHODE: track 0.00 -> 12.5 mm
- net D6-N-CATHODE: track 0.00 -> 11.7 mm
- net D7-N-CATHODE: track 0.00 -> 9.49 mm
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- added copper zone on layer 1, net GND
Other:
- board text added: "cryobondr-rev1-aqc"
