File: meng-spad-quenching/wire-bonding/cryobondr-qbit2.sch (EAGLE design)
At the start: 4 parts

Commit message: Work on cryobondr1 PCB
Parts:
- added IC1: QBIT2-WIREBOND-CRYO1, meng:QBIT2-WIREBOND-CRYO1
- added X1: CONN-D3, meng:MMCX
- added X2: CONN-D5, meng:MMCX
- added X3: CONN-D4, meng:MMCX
- added X4: CONN-D2, meng:MMCX
- added X5: CONN-D1, meng:MMCX
- added X6: CONN-D6, meng:MMCX
- added X7: CONN-D7, meng:MMCX
- added X8: CONN-D8, meng:MMCX
Connections:
- new net D1-N-CATHODE: IC1.D1-N-CATHODE, X5C.1
- new net D1-P-ANODE: IC1.D1-P-ANODE, X5C.GND, X5G.GND@1, X5G.GND@2, X5G.GND@3
- new net D2-N-CATHODE: IC1.D2-N-CATHODE, X4C.1
- new net D2-P-ANODE: IC1.D2-P-ANODE, X4C.GND, X4G.GND@1, X4G.GND@2, X4G.GND@3
- new net D3-N-CATHODE: IC1.D3-N-CATHODE, X1C.1
- new net D3-P-ANODE: IC1.D3-P-ANODE, X1C.GND, X1G.GND@1, X1G.GND@2, X1G.GND@3
- new net D4-N-CATHODE: IC1.D4-N-CATHODE, X3C.1
- new net D4-P-ANODE: IC1.D4-P-ANODE, X3C.GND, X3G.GND@1, X3G.GND@2, X3G.GND@3
- new net D5-N-CATHODE: IC1.D5-N-CATHODE, X2C.1
- new net D5-P-ANODE: IC1.D5-P-ANODE, X2C.GND, X2G.GND@1, X2G.GND@2, X2G.GND@3
- new net D6-N-CATHODE: IC1.D6-N-CATHODE, X6C.1
- new net D6-P-ANODE: IC1.D6-P-ANODE, X6C.GND, X6G.GND@1, X6G.GND@2, X6G.GND@3
- new net D7-N-CATHODE: IC1.D7-N-CATHODE, X7C.1
- new net D7-P-ANODE: IC1.D7-P-ANODE, X7C.GND, X7G.GND@1, X7G.GND@2, X7G.GND@3
- new net D8-N-CATHODE: IC1.D8-N-CATHODE, X8C.1
- new net D8-P-ANODE: IC1.D8-P-ANODE, X8C.GND, X8G.GND@1, X8G.GND@2, X8G.GND@3
Other:
- moved on the sheet: H1, H2, H3, H4
