File: meng-spad-quenching/active-quenching/aqc-rev2-front-panel.sch (EAGLE design)
At the start: 1 part, among them X1 HAMMOND_1455J1201_SIDE_PANEL

Commit message: More work on panel board
Parts:
- added H1: MOUNT-PAD-ROUND3.2, holes:MOUNT-PAD-ROUND3.2
Connections:
- net GND: now also H1.MOUNT
Changed lines of the file:
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@@
 <layers>
 <layer number="1" name="Top" color="4" fill="1" visible="no" active="no"/>
+<layer number="2" name="Route2" color="1" fill="3" visible="no" active="no"/>
+<layer number="3" name="Route3" color="4" fill="3" visible="no" active="no"/>
+<layer number="4" name="Route4" color="1" fill="4" visible="no" active="no"/>
+<layer number="5" name="Route5" color="4" fill="4" visible="no" active="no"/>
+<layer number="6" name="Route6" color="1" fill="8" visible="no" active="no"/>
+<layer number="7" name="Route7" color="4" fill="8" visible="no" active="no"/>
+<layer number="8" name="Route8" color="1" fill="2" visible="no" active="no"/>
+<layer number="9" name="Route9" color="4" fill="2" visible="no" active="no"/>
+<layer number="10" name="Route10" color="1" fill="7" visible="no" active="no"/>
+<layer number="11" name="Route11" color="4" fill="7" visible="no" active="no"/>
+<layer number="12" name="Route12" color="1" fill="5" visible="no" active="no"/>
+<layer number="13" name="Route13" color="4" fill="5" visible="no" active="no"/>
+<layer number="14" name="Route14" color="1" fill="6" visible="no" active="no"/>
+<layer number="15" name="Route15" color="4" fill="6" visible="no" active="no"/>
 <layer number="16" name="Bottom" color="1" fill="1" visible="no" active="no"/>
 <layer number="17" name="Pads" color="2" fill="1" visible="no" active="no"/>
@@
 <part name="X1" library="meng" deviceset="HAMMOND_1455J1201_SIDE_PANEL" device="" value="HAMMOND_1455J1201_SIDE_PANEL"/>
 <part name="GND1" library="supply1" deviceset="GND" device=""/>
+<part name="H1" library="holes" deviceset="MOUNT-PAD-ROUND" device="3.2"/>
 </parts>
 <sheets>
@@
 <instance part="X1" gate="G$1" x="10.16" y="15.24"/>
 <instance part="GND1" gate="1" x="2.54" y="10.16"/>
+<instance part="H1" gate="G$1" x="12.7" y="30.48"/>
 </instances>
 <busses>
@@
 <pinref part="X1" gate="G$1" pin="GND"/>
 <wire x1="2.54" y1="15.24" x2="5.08" y2="15.24" width="0.1524" layer="91"/>
+<wire x1="2.54" y1="15.24" x2="2.54" y2="30.48" width="0.1524" layer="91"/>
+<pinref part="H1" gate="G$1" pin="MOUNT"/>
+<wire x1="2.54" y1="30.48" x2="10.16" y2="30.48" width="0.1524" layer="91"/>
+<junction x="2.54" y="15.24"/>
 </segment>
 </net>
