File: meng-spad-quenching/active-quenching/aqc-rev2.brd (EAGLE design)
At the start: 120 x 74.9 mm, 299 parts, among them IC1 TPS7A4901, IC10 TPS7A3001, IC11 LT1534-1, IC12 74AHC1G04DBV, IC13 74AHC1G04DBV, IC14 NC7WZ16P6X, IC15 LTC1711, IC16 TLV272DGK, IC17 TLV271DBV, IC18 USBLC6-2SC6Y, IC19 ALD1107, IC2 TPS7A4901, IC20 ALD1106, IC21 STM32F411RE, IC22 MAX572X, IC23 TLV271DBV, IC24 LM1117, IC3 LT1534-1, IC4 74AHC1G04DBV, IC5 ADCMP582, IC6 DS1100LU-20+, IC7 74AHC1G04DBV, IC8 NC7SV74K8X, IC9 TLV272DGK, M1 BSS806N, M2 BSS806N, M3 BSS806N, Q1 MMBTH81, Q2 MMBTH81, Q3 MMBTH81, Q4 MMBTH81, Q5 MMBTH81, Q6 IRLML6402TRPBF, SW1 MCU_RST, T1 MMBTH10, T2 MMBTH10, T3 MMBTH10, T4 MMBTH10, T5 MMBTH10, T6 MMBTH10, T7 MMBTH10, U1 MCP4725, U2 SN65EPT22DGK, U3 SN65EPT21DGK, X1 CONN_PULLDN_SENSE, X2 CONN_FORCE_QUENCH, X3 KEYSTONE-7774, X4 CONN_SPAD, X5 CONN_PHOTON_COUNTER, X6 KEYSTONE-7774, X7 CONN_SMU, X8 PN61729-S

Commit message: Fixed component value formatting issues
Parts:
- C16, C53, C81: value 4.7u -> 4u7
- C68: value 33n\ -> 33n
Changed lines of the file:
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@@
 <attribute name="NAME" x="86.0425" y="52.07" size="0.8128" layer="25" font="vector" ratio="16"/>
 </element>
-<element name="C81" library="rcl" package="C0603" value="4.7u" x="82.8675" y="46.6725" smashed="yes" rot="R90">
+<element name="C81" library="rcl" package="C0603" value="4u7" x="82.8675" y="46.6725" smashed="yes" rot="R90">
 <attribute name="NAME" x="83.82" y="47.3075" size="0.8128" layer="25" font="vector" ratio="16"/>
 </element>
@@
 <attribute name="VALUE" x="21.2725" y="54.61" size="0.8128" layer="27" font="vector" ratio="16"/>
 </element>
-<element name="C68" library="rcl" package="C0603" value="33n\" x="101.6" y="37.7825" smashed="yes" rot="R90">
+<element name="C68" library="rcl" package="C0603" value="33n" x="101.6" y="37.7825" smashed="yes" rot="R90">
 <attribute name="NAME" x="100.965" y="40.64" size="0.8128" layer="25" font="vector" ratio="16"/>
 </element>
@@
 <attribute name="NAME" x="90.805" y="40.64" size="0.8128" layer="25" font="vector" ratio="16"/>
 </element>
-<element name="C53" library="rcl" package="C0805" value="4.7u" x="103.8225" y="32.0675" smashed="yes" rot="R270">
+<element name="C53" library="rcl" package="C0805" value="4u7" x="103.8225" y="32.0675" smashed="yes" rot="R270">
 <attribute name="NAME" x="105.0925" y="32.385" size="0.8128" layer="25" font="vector" ratio="16"/>
 </element>
@@
 <attribute name="NAME" x="89.2175" y="44.1325" size="0.8128" layer="25" font="vector" ratio="16"/>
 </element>
-<element name="C16" library="rcl" package="C0805" value="4.7u" x="103.8225" y="12.3825" smashed="yes" rot="R270">
+<element name="C16" library="rcl" package="C0805" value="4u7" x="103.8225" y="12.3825" smashed="yes" rot="R270">
 <attribute name="NAME" x="105.0925" y="12.7" size="0.8128" layer="25" font="vector" ratio="16"/>
 </element>

Commit message: Sorted capacitors by package/value in BOM
Parts:
- C61: value 4.7u -> 4u7
Changed lines of the file:
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@@
 <attribute name="NAME" x="93.0275" y="24.13" size="0.8128" layer="25" font="vector" ratio="16" rot="R180"/>
 </element>
-<element name="C61" library="rcl" package="C0805" value="4.7u" x="83.5025" y="35.8775" smashed="yes" rot="R90">
+<element name="C61" library="rcl" package="C0805" value="4u7" x="83.5025" y="35.8775" smashed="yes" rot="R90">
 <attribute name="NAME" x="84.7725" y="33.9725" size="0.8128" layer="25" font="vector" ratio="16" rot="R180"/>
 </element>

Commit message: Work on BOM
Parts:
- R83, R84: value 100 -> 100R
Changed lines of the file:
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@@
 <attribute name="NAME" x="10.16" y="70.485" size="0.8128" layer="25" font="vector" ratio="16" rot="R180"/>
 </element>
-<element name="R84" library="rcl" package="R0603" value="100" x="11.43" y="69.215" smashed="yes" rot="R270">
+<element name="R84" library="rcl" package="R0603" value="100R" x="11.43" y="69.215" smashed="yes" rot="R270">
 <attribute name="NAME" x="10.4775" y="71.12" size="0.8128" layer="25" font="vector" ratio="16"/>
 </element>
@@
 <attribute name="NAME" x="10.16" y="62.865" size="0.8128" layer="25" font="vector" ratio="16" rot="R180"/>
 </element>
-<element name="R83" library="rcl" package="R0603" value="100" x="11.43" y="61.595" smashed="yes" rot="R270">
+<element name="R83" library="rcl" package="R0603" value="100R" x="11.43" y="61.595" smashed="yes" rot="R270">
 <attribute name="NAME" x="10.4775" y="59.055" size="0.8128" layer="25" font="vector" ratio="16"/>
 </element>

Commit message: Updates to BOM items
Parts:
- R48: value 1k41 -> 1k4
Changed lines of the file:
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@@
 <attribute name="NAME" x="98.425" y="39.37" size="0.8128" layer="25" font="vector" ratio="16"/>
 </element>
-<element name="R48" library="resistor" package="R0603" value="1k41" x="80.9625" y="35.2425" smashed="yes" rot="R90">
+<element name="R48" library="resistor" package="R0603" value="1k4" x="80.9625" y="35.2425" smashed="yes" rot="R90">
 <attribute name="NAME" x="79.9465" y="40.0685" size="0.8128" layer="25" font="vector" ratio="16" rot="R180"/>
 </element>

Commit message: Started new PCB for box front panel
Parts:
- C66: value 1n -> 470p
- R43, R59: value 49R9 -> 200R
- R46, R49: value 49R9 -> 100R
Changed lines of the file:
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@@
 <attribute name="NAME" x="55.5625" y="39.0525" size="0.8128" layer="25" font="vector" ratio="16"/>
 </element>
-<element name="C66" library="rcl" package="C0603" value="1n" x="50.95875" y="37.7825" smashed="yes" rot="R90">
+<element name="C66" library="rcl" package="C0603" value="470p" x="50.95875" y="37.7825" smashed="yes" rot="R90">
 <attribute name="NAME" x="51.91125" y="36.5125" size="0.8128" layer="25" font="vector" ratio="16"/>
 </element>
@@
 <attribute name="NAME" x="24.13" y="41.275" size="0.8128" layer="25" font="vector" ratio="16"/>
 </element>
-<element name="R49" library="rcl" package="R0603" value="49R9" x="21.9075" y="36.5125" smashed="yes" rot="R90">
+<element name="R49" library="rcl" package="R0603" value="100R" x="21.9075" y="36.5125" smashed="yes" rot="R90">
 <attribute name="NAME" x="20.955" y="37.465" size="0.8128" layer="25" font="vector" ratio="16" rot="R180"/>
 </element>
-<element name="R59" library="rcl" package="R0603" value="49R9" x="26.9875" y="42.2275" smashed="yes" rot="R180">
+<element name="R59" library="rcl" package="R0603" value="200R" x="26.9875" y="42.2275" smashed="yes" rot="R180">
 <attribute name="NAME" x="28.8925" y="42.2275" size="0.8128" layer="25" font="vector" ratio="16"/>
 </element>
-<element name="R46" library="rcl" package="R0603" value="49R9" x="21.9075" y="33.3375" smashed="yes" rot="R90">
+<element name="R46" library="rcl" package="R0603" value="100R" x="21.9075" y="33.3375" smashed="yes" rot="R90">
 <attribute name="NAME" x="20.955" y="33.3375" size="0.8128" layer="25" font="vector" ratio="16" rot="R180"/>
 </element>
-<element name="R43" library="rcl" package="R0603" value="49R9" x="28.575" y="31.115" smashed="yes">
+<element name="R43" library="rcl" package="R0603" value="200R" x="28.575" y="31.115" smashed="yes">
 <attribute name="NAME" x="30.48" y="30.7975" size="0.8128" layer="25" font="vector" ratio="16"/>
 </element>

Commit message: Made & exported modulator switch board
Parts:
- R56, R65: value 470R -> 220R
Changed lines of the file:
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@@
 <attribute name="NAME" x="18.0975" y="24.13" size="0.8128" layer="25" font="vector" ratio="16" rot="R180"/>
 </element>
-<element name="R56" library="rcl" package="R0603" value="470R" x="31.75" y="39.6875" smashed="yes" rot="R90">
+<element name="R56" library="rcl" package="R0603" value="220R" x="31.75" y="39.6875" smashed="yes" rot="R90">
 <attribute name="NAME" x="30.7975" y="42.545" size="0.8128" layer="25" font="vector" ratio="16"/>
 </element>
@@
 <attribute name="NAME" x="32.7025" y="48.26" size="0.8128" layer="25" font="vector" ratio="16"/>
 </element>
-<element name="R65" library="rcl" package="R0603" value="470R" x="39.0525" y="46.6725" smashed="yes" rot="R180">
+<element name="R65" library="rcl" package="R0603" value="220R" x="39.0525" y="46.6725" smashed="yes" rot="R180">
 <attribute name="NAME" x="40.9575" y="49.53" size="0.8128" layer="25" font="vector" ratio="16"/>
 </element>
