File: meng-plant-raman/leaf-heater-controller-rev1.sch (EAGLE design)
At the start: 0 parts

Commit message: Updated leaf heaters with 6-pin JST SH
Parts:
- added C1: 100n, rcl-modified-footprints:C-EUC0603
- added R1, R2: 2k2, rcl-modified-footprints:R-EU_R0603
- added TP1: 105-0752-001, meng-plant-raman:CINCH-BANANA
- added TP2: 105-0753-001, meng-plant-raman:CINCH-BANANA
- added U1: ARDUINOR3-DIMENSION, adafruit:ARDUINOR3-DIMENSION
- added X1, X2: SM06B-SRSS-TB, meng-plant-raman:JST-SH-6PIN
Connections:
- new net GND: C1.2, X1.5, X1.PAD1, X1.PAD2, X2.2, X2.PAD1, X2.PAD2
- new net HEATER_GND: TP2.BANANA, X1.6, X2.1
- new net HEATER_VDD: TP1.BANANA, X1.1, X2.6
- new net PP_P3V3_SENSOR: C1.1, R1.2, R2.2, U1.3V, X1.4, X2.3
- new net TEMP_SCL: R1.1, U1.SCL, X1.3, X2.4
- new net TEMP_SDA: R2.1, U1.SDA, X1.2, X2.5

Commit message: Updates to component selection
Other:
- note added: "Mates to: 105-0772-001"
- note added: "Mates to: 105-0773-001"
Changed lines of the file:
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@@
 <sheet>
 <plain>
+<text x="246.38" y="147.32" size="1.778" layer="98">Mates to:
+105-0772-001</text>
+<text x="246.38" y="124.46" size="1.778" layer="98">Mates to:
+105-0773-001</text>
 </plain>
 <instances>
@@
 </drawing>
 <compatibility>
+<note version="6.3" minversion="6.2.2" severity="warning">
+Since Version 6.2.2 text objects can contain more than one line,
+which will not be processed correctly with this version.
+</note>
 <note version="8.2" severity="warning">
 Since Version 8.2, EAGLE supports online libraries. The ids
