File: meng-plant-raman/leaf-heater-controller-rev2.brd (EAGLE design)
At the start: 68.6 x 53.3 mm, 15 parts, among them U1 ARDUINOR3-DIMENSION, U2 OPA2333, X1 SM06B-SRSS-TB, X2 SM06B-SRSS-TB

Commit message: Fixed one-shot error, layout done
Parts:
- C1: value 100p -> CAP CER 100PF 50V C0G/NP0 0603
- C2, C3: value 100n -> CAP CER 0.1UF 16V X7R 0603
- R1: value 10k -> RES SMD 10K OHM 1% 1/16W 0603
- R2: value 10R -> RES SMD 10 OHM 1% 1/16W 0603
- R3: value 3R3 -> RES SMD 0.33 OHM 1% 1W 1210
- R4, R5: value 2k2 -> RES SMD 2.2K OHM 1% 1/16W 0603
