File: isg-clock-generator-rev1/isg-clock-generator-rev1.sch (EAGLE design)
At the start: 68 parts, among them IC1 LMK03318RHSR, X1 OUT0_P, X2 OUT0_N, X3 OUT1_P, X4 OUT1_N

Commit message: More progress idk
Parts:
- removed JP1: (no value), jumper:JP5Q
- added C44, C45, C49, C50: CAP CER 10000PF 25V X7R 0603 10%, rcl-modified-footprints:C-EUC0603
- added C46, C48, C51, C53: CAP CER 0.1UF 25V X7R 0603 10%, rcl-modified-footprints:C-EUC0603
- added C47, C52: CAP CER 10UF 16V X7R 0805 20%, rcl:C-EUC0805
- added C54: CAP CER 0.01uF X7R 0402, rcl-modified-footprints:C-EUC0402
- added C55: CAP CER 22uF 6.3V 0603, rcl-modified-footprints:C-EUC0603
- added C56: CAP CER 0.033uF 0603, rcl-modified-footprints:C-EUC0603
- added C57: CAP CER 3300pF 0603, rcl-modified-footprints:C-EUC0603
- added C58, C62, C63: DNP, rcl-modified-footprints:C-EUC0603
- added C59, C60: 0R JUMPER, rcl-modified-footprints:C-EUC0603
- added C61: DNP, rcl-modified-footprints:C-EUC0402
- added IC2, IC3: TPS7A4901, Kramnik's Library:TPS7A
- added JP10: RSEL, isg-clock-generator:JP2E
- added JP11: (no value), jumper:JP8Q
- added JP12: (no value), jumper:JP3Q
- added JP13: PRIREF_VCM, jumper:JP2E
- added JP14: CON_OST_302-S101, Kramnik's Library:CON_OST_302-S101
- added JP2: STAT_LED_EN, jumper:JP1Q
- added JP3: GPIO5, isg-clock-generator:JP2E
- added JP4: GPIO4, isg-clock-generator:JP2E
- added JP5: GPIO3, isg-clock-generator:JP2E
- added JP6: GPIO2, isg-clock-generator:JP2E
- added JP7: GPIO1, isg-clock-generator:JP2E
- added JP8: GPIO0, isg-clock-generator:JP2E
- added JP9: HWCTRL, isg-clock-generator:JP2E
- added R10, R14: RES SMD 76.8K OHM 1% 1/10W 0603, rcl-modified-footprints:R-EU_R0603
- added R11, R12, R13, R26, R28, R29, R41, R42, R44, R45, R49, R50, R51, R52, R53, R6, R8, R9: DNP, rcl-modified-footprints:R-EU_R0603
- added R15, R17, R18, R7: RES SMD 24K OHM 1% 1/10W 0603, rcl-modified-footprints:R-EU_R0603
- added R16, R27, R30, R33, R36, R40, R43: RES SMD 1K OHM 1% 1/10W 0603, rcl-modified-footprints:R-EU_R0603
- added R19: RES SMD 0 OHM 1% 1/10W 0603, rcl-modified-footprints:R-EU_R0603
- added R20: RES SMD 2.32K OHM 1% 1/10W 0603, rcl-modified-footprints:R-EU_R0603
- added R21: RES SMD 5.62K OHM 1% 1/10W 0603, rcl-modified-footprints:R-EU_R0603
- added R22: RES SMD 10.5K OHM 1% 1/10W 0603, rcl-modified-footprints:R-EU_R0603
- added R23: RES SMD 18.7K OHM 1% 1/10W 0603, rcl-modified-footprints:R-EU_R0603
- added R24: RES SMD 34.8K OHM 1% 1/10W 0603, rcl-modified-footprints:R-EU_R0603
- added R25: RES SMD 84.5K OHM 1% 1/10W 0603, rcl-modified-footprints:R-EU_R0603
- added R3, R4, R46, R47, R48, R5: 0R JUMPER 0603, rcl-modified-footprints:R-EU_R0603
- added R31, R34, R37, R39: RES SMD 13.0K OHM 1% 1/10W 0603, rcl-modified-footprints:R-EU_R0603
- added R32, R35, R38: RES SMD 4.99K OHM 1% 1/10W 0603, rcl-modified-footprints:R-EU_R0603
- added X5: OUT1_P, con-coax:SMA-142-0701-881/886
- Q1: value (none) -> 7M50072001
- R1, R2: value 510 -> RES SMD 510R 0603
- X3: value OUT1_P -> OUT2_P
- X4: value OUT1_N -> OUT1_P
Connections:
- net LF2 renamed NC_PIN
- net N$17 renamed STATUS0
- net N$18 renamed STATUS1
- removed net N$15: IC1.SECREF_P
- removed net N$16: IC1.PRIREF_N
- removed net N$19: IC1.PRIREF_P
- removed net NC_OUT2_P: IC1.OUT2_P
- removed net OUT1_N: IC1.OUT1_N, X4.1
- removed net OUT1_P: IC1.OUT1_P, X3.1
- new net GPIO5_SEL_11_12: JP11.12, R24.2
- new net GPIO5_SEL_13_14: JP11.14, R25.2
- new net GPIO5_SEL_15_16: JP11.16, R26.2
- new net GPIO5_SEL_1_2: JP11.2, R19.2
- new net GPIO5_SEL_3_4: JP11.4, R20.2
- new net GPIO5_SEL_5_6: JP11.6, R21.2
- new net GPIO5_SEL_7_8: JP11.8, R22.2
- new net GPIO5_SEL_9_10: JP11.10, R23.2
- new net LDO_P3V3_SS: C44.1, C49.1, IC2.NR/SS, IC3.NR/SS
- new net LDO_P5V0_FB_CH1: C45.2, C50.2, IC2.FB, IC3.FB, R10.1, R14.1, R15.1, R7.1
- new net N$1: R6.2, R8.2, R9.2
- new net N$10: JP14.3
- new net N$11: JP14.1
- new net N$12: JP14.8
- new net N$13: JP14.4
- new net N$22: C55.1, JP12.5
- new net N$23: C56.1, JP12.3
- new net N$24: JP4.2, R27.1
- new net N$25: JP5.2, R30.1
- new net N$26: JP8.2, R39.1
- new net N$27: JP6.2, R33.1
- new net N$28: JP9.2, R40.1
- new net N$29: JP7.2, R36.1
- new net N$30: C57.1, JP12.1
- new net N$31: JP10.2, R43.1
- new net N$32: JP12.2, JP12.4, JP12.6, R46.2
- new net N$4: JP3.3, R16.1
- new net N$5: JP13.3, R51.1, R52.2
- new net N$6: JP14.5, R53.1
- new net NC_OUT1_N: IC1.OUT1_N
- new net NC_OUT1_P: IC1.OUT1_P
- new net OUT0_R_N: R12.2, R4.1, R8.1, X2.1
- new net OUT0_R_P: R11.2, R3.1, R6.1, X1.1
- new net OUT2_P: IC1.OUT2_P, R5.2
- new net OUT2_R_P: R13.2, R5.1, R9.1, X3.1
- new net PP_P1V8_VDDO: C26.1, C30.1, C34.1, C38.1, C42.1, C45.1, C46.1, C47.1, C6.1, IC2.OUT, L1.P$2, L10.P$2, L6.P$2, L7.P$2, L8.P$2, L9.P$2, R10.2
- new net PP_P3V3_PLL_CORE: C20.1, C21.1, C22.1, C23.1, C50.1, C51.1, C52.1, IC3.OUT, JP10.3, JP2.2, JP4.3, JP5.3, JP6.3, JP7.3, JP8.3, JP9.3, L2.P$1, L3.P$1, L4.P$1, L5.P$1, R14.2, R16.2, R17.1, R28.2, R31.2, R34.2, R37.2, R41.2, R44.2, R51.2, R53.2
- new net PRIREF_N: IC1.PRIREF_N, R48.1, R50.2
- new net PRIREF_P: IC1.PRIREF_P, R47.1, R49.2
- new net PRIREF_RC_N: C60.1, X5.1
- new net PRIREF_RC_P: C59.1, X4.1
- new net PRIREF_R_N: C60.2, R48.2
- new net PRIREF_R_P: C59.2, R47.2
- new net PRIREF_VCM: C61.1, JP13.2, R49.1, R50.1
- new net SECREF_N: C62.1, IC1.SECREF_N, Q1.1
- new net SECREF_P: C63.1, IC1.SECREF_P, Q1.2
- new net STATUS_LED_PWR: JP2.1, R1.2, R2.2
- new net VIN: C48.1, C53.1, IC2.IN, IC3.IN, R18.1
- net GND: now also C44.2, C46.2, C47.2, C48.2, C49.2, C51.2, C52.2, C53.2, C54.2, C55.2, C56.2, C57.2, C58.2, C61.2, C62.2, C63.2, IC2.GND, IC3.GND, JP10.1, JP11.1, JP11.11, JP11.13, JP11.15, JP11.3, JP11.5, JP11.7, JP11.9, JP13.1, JP14.6, JP3.1, JP4.1, JP5.1, JP6.1, JP7.1, JP8.1, JP9.1, R11.1, R12.1, R13.1, R15.2, R29.1, R32.1, R35.1, R38.1, R42.1, R45.1, R52.1, R7.2, X5.2
- net GPIO0: now also R39.2
- net GPIO1: now also R36.2, R37.1, R38.2
- net GPIO2: now also R33.2, R34.1, R35.2
- net GPIO3: now also R30.2, R31.1, R32.2
- net GPIO4: now also R27.2, R28.1, R29.2
- net GPIO5: now also JP3.2, R19.1, R20.1, R21.1, R22.1, R23.1, R24.1, R25.1, R26.1
- net HW_SW_CTRL: now also R40.2, R41.1, R42.2
- net LF1: now also C58.1, R46.1
- net N$14: now also JP14.2; no longer IC1.SECREF_N
- net N$2: now also IC2.EN, R17.2; no longer C20.1, C21.1, C22.1, C23.1, L2.P$1, L3.P$1, L4.P$1, L5.P$1
- net N$3: now also IC3.EN, R18.2; no longer C26.1, C30.1, C34.1, C38.1, C42.1, C6.1, L1.P$2, L10.P$2, L6.P$2, L7.P$2, L8.P$2, L9.P$2
- net N$9: now also JP14.7; no longer R1.2, R2.2
- net OUT0_N: now also R4.2; no longer X2.1
- net OUT0_P: now also R3.2; no longer X1.1
- net PDN: now also C54.1
- net REFSEL: now also R43.2, R44.1, R45.2
- net SCL: now also JP14.9
- net SDA: now also JP14.10
Other:
- note added: "1-2 = INT-N 3-4 = FRAC-N 5-6 = NARROW"
- note added: "All feedback resistors 1% or better"
- note added: "Diff. clock"
- note added: "For Core -> Output power sequenching V_EN(HIGH) = 2.1V"
- note added: "I2C to TI USB2ANY connector"
- note added: "Internal 200k pullup to VDDO_01"
- note added: "JP Pins: 1-2 = High Open = Mid 2-3 = Low"
- note added: "LF = Loop Filter"
- note added: "Optional VCM refs"
- note added: "SE clock"
- note added: "TI USB2ANY connector"
- note added: "TPS7A4901 (Positive)"
- note added: "TPS7A4901: 150mA Max. This might be insufficient!!! TODO: switch to TPS7A8001"
- note added: "Vout/(Rtop+Rbottom) > 5uA"
- note added: "Vref = 1.188V Nominal"
- note added: "Vref(1+Rtop/Rbottom) = Vout"
- note added: "XTAL: SecRef only Todo: get symbol with grounded pads"
- note removed: "To TI USB2ANY connector"
- note removed: "XTAL: SecRef only"
- moved on the sheet: C1, C10, C11, C12, C13, C14, C15, C16, C17, C18, C19, C2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

Commit message: Started decap placement
Parts:
- IC1: device isg-clock-generator:LMK03318RHSR -> isg-clock-generator:LMK03318RHSRRHS0048A_NV
- X4: value OUT1_P -> PRIREF_P
- X5: value OUT1_P -> PRIREF_N
Changed lines of the file:
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@@
 </classes>
 <parts>
-<part name="IC1" library="isg-clock-generator" deviceset="LMK03318RHSR" device=""/>
+<part name="IC1" library="isg-clock-generator" deviceset="LMK03318RHSR" device="RHS0048A_NV" value="LMK03318RHSR"/>
 <part name="X1" library="con-coax" library_urn="urn:adsk.eagle:library:133" deviceset="SMA-" device="142-0701-881/886" package3d_urn="urn:adsk.eagle:package:6216/1" value="OUT0_P"/>
 <part name="X2" library="con-coax" library_urn="urn:adsk.eagle:library:133" deviceset="SMA-" device="142-0701-881/886" package3d_urn="urn:adsk.eagle:package:6216/1" value="OUT0_N"/>
@@
 <part name="DNP44" library="meng" deviceset="ARROW_1DIR" device=""/>
 <part name="DNP45" library="meng" deviceset="ARROW_1DIR" device=""/>
-<part name="X4" library="con-coax" library_urn="urn:adsk.eagle:library:133" deviceset="SMA-" device="142-0701-881/886" package3d_urn="urn:adsk.eagle:package:6216/1" value="OUT1_P"/>
-<part name="X5" library="con-coax" library_urn="urn:adsk.eagle:library:133" deviceset="SMA-" device="142-0701-881/886" package3d_urn="urn:adsk.eagle:package:6216/1" value="OUT1_P"/>
+<part name="X4" library="con-coax" library_urn="urn:adsk.eagle:library:133" deviceset="SMA-" device="142-0701-881/886" package3d_urn="urn:adsk.eagle:package:6216/1" value="PRIREF_P"/>
+<part name="X5" library="con-coax" library_urn="urn:adsk.eagle:library:133" deviceset="SMA-" device="142-0701-881/886" package3d_urn="urn:adsk.eagle:package:6216/1" value="PRIREF_N"/>
 <part name="GND80" library="supply1" library_urn="urn:adsk.eagle:library:371" deviceset="GND" device=""/>
 <part name="GND81" library="supply1" library_urn="urn:adsk.eagle:library:371" deviceset="GND" device=""/>

Commit message: Fit all components on board except power supplies (need to swap LDO part)
Parts:
- JP13: device jumper:JP2E -> isg-clock-generator:JP2E
Other:
- note added: "TODO: FIX INDUCTOR PACKAGES"
Changed lines of the file:
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@@
 <part name="C61" library="rcl-modified-footprints" deviceset="C-EU" device="C0402" package3d_urn="urn:adsk.eagle:package:23626/1" value="DNP"/>
 <part name="GND82" library="supply1" library_urn="urn:adsk.eagle:library:371" deviceset="GND" device=""/>
-<part name="JP13" library="jumper" library_urn="urn:adsk.eagle:library:252" deviceset="JP2E" device="" package3d_urn="urn:adsk.eagle:package:15452/1" value="PRIREF_VCM"/>
+<part name="JP13" library="isg-clock-generator" deviceset="JP2E" device="" value="PRIREF_VCM"/>
 <part name="GND83" library="supply1" library_urn="urn:adsk.eagle:library:371" deviceset="GND" device=""/>
 <part name="C62" library="rcl-modified-footprints" deviceset="C-EU" device="C0603" package3d_urn="urn:adsk.eagle:package:23616/2" value="DNP"/>
@@
 3-4 = FRAC-N
 5-6 = NARROW</text>
+<text x="236.22" y="314.96" size="1.778" layer="98">TODO: FIX INDUCTOR PACKAGES</text>
 </plain>
 <instances>

Commit message: Updated LDOs for 1A, all parts roughly placed in layout, power input TODO
Parts:
- removed C50: CAP CER 10000PF 25V X7R 0603 10%, rcl-modified-footprints:C-EUC0603
- removed C52: CAP CER 10UF 16V X7R 0805 20%, rcl:C-EUC0805
- removed IC2, IC3: TPS7A4901, Kramnik's Library:TPS7A
- added IC4, IC5: TPS7A8001DRBR, isg-clock-generator:TPS7A8001DRBR
- added JP1: MOTHERBOARD, isg-clock-generator:JP5Q
- added X6: 22-23-2021, con-molex:22-23-2021
- C45: value CAP CER 10000PF 25V X7R 0603 10% -> CAP CER 4.7UF 6.3V X5R 0603 10%
- C47: value CAP CER 10UF 16V X7R 0805 20% -> CAP CER 4.7UF 6.3V X5R 0603 10%; device rcl:C-EUC0805 -> rcl-modified-footprints:C-EUC0603
- C61: value DNP -> DNP 0603; device rcl-modified-footprints:C-EUC0402 -> rcl-modified-footprints:C-EUC0603
- JP11: value (none) -> XO_MARGIN; device jumper:JP8Q -> isg-clock-generator:JP8Q
- JP12: value (none) -> LOOP_FILTER; device jumper:JP3Q -> isg-clock-generator:JP3Q
- R10, R14: value RES SMD 76.8K OHM 1% 1/10W 0603 -> RES SMD 4.99K OHM 1% 1/10W 0603
- R15: value RES SMD 24K OHM 1% 1/10W 0603 -> RES SMD 1.62K OHM 1% 1/10W 0603
- R17, R18: value RES SMD 24K OHM 1% 1/10W 0603 -> RES SMD 4.99K OHM 1% 1/10W 0603
- R51, R52: value DNP -> DNP 0603
- R7: value RES SMD 24K OHM 1% 1/10W 0603 -> RES SMD 3.92K OHM 1% 1/10W 0603
Connections:
- net N$22 renamed LF_NARROW
- net N$23 renamed LF_FRAC_N
- net N$30 renamed LF_INT_N\
- net N$32 renamed LF_R
- removed net LDO_P3V3_SS: C44.1, C49.1, IC2.NR/SS, IC3.NR/SS
- removed net LDO_P5V0_FB_CH1: C45.2, C50.2, IC2.FB, IC3.FB, R10.1, R14.1, R15.1, R7.1
- removed net N$2: IC2.EN, R17.2
- removed net N$3: IC3.EN, R18.2
- new net LDO_PVCORE_EN: IC4.EN, R18.2
- new net LDO_PVCORE_FB: IC4.FB/SNS, R14.1, R15.1
- new net LDO_PVCORE_SS: C49.1, IC4.NR/SS
- new net LDO_PVDDIO_EN: IC5.EN, R17.2
- new net LDO_PVDDIO_FB: IC5.FB/SNS, R10.1, R7.1
- new net LDO_PVDDIO_SS: C44.1, IC5.NR/SS
- net GND: now also C45.2, IC4.GND, IC5.GND; no longer C52.2, IC2.GND, IC3.GND
- net PP_P1V8_VDDO: now also IC5.OUT, IC5.OUT_2; no longer C45.1, IC2.OUT
- net PP_P3V3_PLL_CORE: now also C45.1, IC4.OUT, IC4.OUT_2; no longer C50.1, C52.1, IC3.OUT
- net VIN: now also IC4.IN, IC4.IN_2, IC5.IN, IC5.IN_2; no longer IC2.IN, IC3.IN
Other:
- note added: "EN resistor values should be on the order of 1s to 10s of kOhms."
- note added: "Headers for Connecting to Motherboard"
- note added: "TODO: figure out power input connectors"
- note added: "TODO: fix all values for new LDO MPN"
- note added: "Vref = 0.8V Nominal"
- note removed: "TPS7A4901 (Positive)"
- note removed: "TPS7A4901: 150mA Max. This might be insufficient!!! TODO: switch to TPS7A8001"
- note removed: "Vout/(Rtop+Rbottom) > 5uA"
- note removed: "Vref = 1.188V Nominal"
- moved on the sheet: C45, C46, C47, C48, C51, C53, R10, R14, R15, R17, R18, R7

Commit message: Started working on routing
Parts:
- JP10: value RSEL -> REFSEL
- R40: value RES SMD 1K OHM 1% 1/10W 0603 -> RES SMD 10K OHM 1% 1/10W 0603
- X6: value 22-23-2021 -> V_INPUT
Connections:
- net GND: now also JP1.3, JP1.4, JP1.6
- net HW_SW_CTRL: now also JP1.8
- net SCL: now also JP1.10
- net SDA: now also JP1.9
- net STATUS0: now also JP1.7
- net STATUS1: now also JP1.5
- net VIN: now also JP1.1, JP1.2
Changed lines of the file:
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@@
 <part name="JP9" library="isg-clock-generator" deviceset="JP2E" device="" value="HWCTRL"/>
 <part name="GND72" library="supply1" library_urn="urn:adsk.eagle:library:371" deviceset="GND" device=""/>
-<part name="R40" library="rcl-modified-footprints" deviceset="R-EU_" device="R0603" package3d_urn="urn:adsk.eagle:package:23555/2" value="RES SMD 1K OHM 1% 1/10W 0603"/>
+<part name="R40" library="rcl-modified-footprints" deviceset="R-EU_" device="R0603" package3d_urn="urn:adsk.eagle:package:23555/2" value="RES SMD 10K OHM 1% 1/10W 0603"/>
 <part name="R41" library="rcl-modified-footprints" deviceset="R-EU_" device="R0603" package3d_urn="urn:adsk.eagle:package:23555/2" value="DNP"/>
 <part name="R42" library="rcl-modified-footprints" deviceset="R-EU_" device="R0603" package3d_urn="urn:adsk.eagle:package:23555/2" value="DNP"/>
 <part name="GND73" library="supply1" library_urn="urn:adsk.eagle:library:371" deviceset="GND" device=""/>
-<part name="JP10" library="isg-clock-generator" deviceset="JP2E" device="" value="RSEL"/>
+<part name="JP10" library="isg-clock-generator" deviceset="JP2E" device="" value="REFSEL"/>
 <part name="GND74" library="supply1" library_urn="urn:adsk.eagle:library:371" deviceset="GND" device=""/>
 <part name="R43" library="rcl-modified-footprints" deviceset="R-EU_" device="R0603" package3d_urn="urn:adsk.eagle:package:23555/2" value="RES SMD 1K OHM 1% 1/10W 0603"/>
@@
 <part name="IC5" library="isg-clock-generator" deviceset="TPS7A8001DRBR" device="" value="TPS7A8001DRBR"/>
 <part name="JP1" library="isg-clock-generator" deviceset="JP5Q" device="" package3d_urn="urn:adsk.eagle:package:15454/1" value="MOTHERBOARD"/>
-<part name="X6" library="con-molex" library_urn="urn:adsk.eagle:library:165" deviceset="22-23-2021" device="" package3d_urn="urn:adsk.eagle:package:8078633/1"/>
+<part name="X6" library="con-molex" library_urn="urn:adsk.eagle:library:165" deviceset="22-23-2021" device="" package3d_urn="urn:adsk.eagle:package:8078633/1" value="V_INPUT"/>
 <part name="C45" library="rcl-modified-footprints" deviceset="C-EU" device="C0603" package3d_urn="urn:adsk.eagle:package:23616/2" value="CAP CER 4.7UF 6.3V X5R 0603 10%"/>
 <part name="C47" library="rcl-modified-footprints" deviceset="C-EU" device="C0603" package3d_urn="urn:adsk.eagle:package:23616/2" value="CAP CER 4.7UF 6.3V X5R 0603 10%"/>
+<part name="DNP58" library="meng" deviceset="ARROW_1DIR" device=""/>
+<part name="DNP59" library="meng" deviceset="ARROW_1DIR" device=""/>
+<part name="GND88" library="supply1" deviceset="GND" device=""/>
+<part name="U$4" library="Kramnik's Library" deviceset="LEFT_ARROW" device=""/>
 </parts>
 <sheets>
@@
 <text x="236.22" y="314.96" size="1.778" layer="98">TODO: FIX INDUCTOR PACKAGES</text>
 <text x="124.46" y="416.56" size="1.778" layer="98">TODO: fix all values for new LDO MPN</text>
-<text x="312.42" y="414.02" size="3.81" layer="98">Headers for Connecting to Motherboard </text>
+<text x="312.42" y="416.56" size="3.81" layer="98">Headers for Connecting to Motherboard </text>
 <text x="15.24" y="416.56" size="1.778" layer="98">TODO: figure out power input connectors</text>
 <text x="86.36" y="335.28" size="1.27" layer="98">Vref(1+Rtop/Rbottom) = Vout</text>
@@
 </instance>
 <instance part="JP1" gate="B" x="353.06" y="396.24" smashed="yes" rot="R270">
-<attribute name="NAME" x="347.98" y="403.86" size="1.778" layer="95"/>
-<attribute name="VALUE" x="347.98" y="386.715" size="1.778" layer="96"/>
+<attribute name="NAME" x="347.98" y="411.48" size="1.778" layer="95"/>
+<attribute name="VALUE" x="347.98" y="409.575" size="1.778" layer="96"/>
 </instance>
 <instance part="X6" gate="-1" x="20.32" y="378.46" smashed="yes" rot="R180">
@@
 <attribute name="VALUE" x="169.164" y="338.201" size="0.8128" layer="96"/>
 </instance>
+<instance part="DNP58" gate="G$1" x="78.74" y="144.78" smashed="yes"/>
+<instance part="DNP59" gate="G$1" x="83.82" y="139.7" smashed="yes" rot="R90"/>
+<instance part="GND88" gate="1" x="342.9" y="378.46" smashed="yes">
+<attribute name="VALUE" x="340.36" y="375.92" size="1.778" layer="96"/>
+</instance>
+<instance part="U$4" gate="G$1" x="337.82" y="408.94" smashed="yes" rot="R180"/>
 </instances>
 <busses>
@@
 <wire x1="350.52" y1="40.64" x2="347.98" y2="40.64" width="0.1524" layer="91"/>
 </segment>
+<segment>
+<pinref part="GND88" gate="1" pin="GND"/>
+<wire x1="342.9" y1="381" x2="342.9" y2="383.54" width="0.1524" layer="91"/>
+<pinref part="JP1" gate="B" pin="3"/>
+<wire x1="342.9" y1="383.54" x2="342.9" y2="398.78" width="0.1524" layer="91"/>
+<wire x1="342.9" y1="398.78" x2="345.44" y2="398.78" width="0.1524" layer="91"/>
+<pinref part="JP1" gate="B" pin="4"/>
+<wire x1="360.68" y1="398.78" x2="363.22" y2="398.78" width="0.1524" layer="91"/>
+<wire x1="363.22" y1="398.78" x2="363.22" y2="396.24" width="0.1524" layer="91"/>
+<wire x1="363.22" y1="396.24" x2="363.22" y2="383.54" width="0.1524" layer="91"/>
+<wire x1="363.22" y1="383.54" x2="342.9" y2="383.54" width="0.1524" layer="91"/>
+<junction x="342.9" y="383.54"/>
+<pinref part="JP1" gate="B" pin="6"/>
+<wire x1="360.68" y1="396.24" x2="363.22" y2="396.24" width="0.1524" layer="91"/>
+<junction x="363.22" y="396.24"/>
+</segment>
 </net>
 <net name="DECAP_LDO" class="0">
@@
 <label x="360.68" y="35.56" size="1.778" layer="95"/>
 </segment>
+<segment>
+<pinref part="JP1" gate="B" pin="9"/>
+<wire x1="345.44" y1="391.16" x2="332.74" y2="391.16" width="0.1524" layer="91"/>
+<label x="332.74" y="391.16" size="1.778" layer="95" rot="R180"/>
+</segment>
 </net>
 <net name="SCL" class="0">
@@
 <wire x1="332.74" y1="35.56" x2="320.04" y2="35.56" width="0.1524" layer="91"/>
 <label x="320.04" y="35.56" size="1.778" layer="95" rot="R180"/>
+</segment>
+<segment>
+<pinref part="JP1" gate="B" pin="10"/>
+<wire x1="360.68" y1="391.16" x2="375.92" y2="391.16" width="0.1524" layer="91"/>
+<label x="375.92" y="391.16" size="1.778" layer="95"/>
 </segment>
 </net>
@@
 <label x="378.46" y="118.11" size="0.8128" layer="95" rot="R180"/>
 </segment>
+<segment>
+<pinref part="JP1" gate="B" pin="7"/>
+<wire x1="345.44" y1="393.7" x2="332.74" y2="393.7" width="0.1524" layer="91"/>
+<label x="332.74" y="393.7" size="1.778" layer="95" rot="R180"/>
+</segment>
 </net>
 <net name="STATUS1" class="0">
@@
 <wire x1="426.72" y1="114.3" x2="426.72" y2="119.38" width="0.1524" layer="91"/>
 <label x="378.46" y="115.57" size="0.8128" layer="95" rot="R180"/>
+</segment>
+<segment>
+<pinref part="JP1" gate="B" pin="5"/>
+<wire x1="345.44" y1="396.24" x2="332.74" y2="396.24" width="0.1524" layer="91"/>
+<label x="332.74" y="396.24" size="1.778" layer="95" rot="R180"/>
 </segment>
 </net>
@@
 <junction x="78.74" y="355.6"/>
 </segment>
+<segment>
+<pinref part="JP1" gate="B" pin="1"/>
+<wire x1="345.44" y1="401.32" x2="342.9" y2="401.32" width="0.1524" layer="91"/>
+<wire x1="342.9" y1="401.32" x2="342.9" y2="406.4" width="0.1524" layer="91"/>
+<wire x1="342.9" y1="406.4" x2="342.9" y2="408.94" width="0.1524" layer="91"/>
+<wire x1="342.9" y1="408.94" x2="332.74" y2="408.94" width="0.1524" layer="91"/>
+<wire x1="342.9" y1="406.4" x2="363.22" y2="406.4" width="0.1524" layer="91"/>
+<junction x="342.9" y="406.4"/>
+<wire x1="363.22" y1="406.4" x2="363.22" y2="401.32" width="0.1524" layer="91"/>
+<pinref part="JP1" gate="B" pin="2"/>
+<wire x1="363.22" y1="401.32" x2="360.68" y2="401.32" width="0.1524" layer="91"/>
+<label x="332.74" y="408.94" size="1.778" layer="95" rot="R180"/>
+</segment>
 </net>
 <net name="LDO_PVDDIO_FB" class="0">
@@
 <label x="312.42" y="146.05" size="0.8128" layer="95" rot="R180"/>
 <wire x1="83.82" y1="144.78" x2="314.96" y2="144.78" width="0.1524" layer="91"/>
-</segment>
-</net>
+<wire x1="83.82" y1="144.78" x2="73.66" y2="144.78" width="0.1524" layer="91"/>
+<junction x="83.82" y="144.78"/>
+<label x="73.66" y="144.78" size="1.778" layer="95" rot="R180"/>
+</segment>
+<segment>
+<pinref part="JP1" gate="B" pin="8"/>
+<wire x1="360.68" y1="393.7" x2="375.92" y2="393.7" width="0.1524" layer="91"/>
+<label x="375.92" y="393.7" size="1.778" layer="95"/>
+</segment>
+</net>

Commit message: First-pass routing of high speed output signals
Parts:
- added C50, C52, C64: 0R JUMPER, rcl-modified-footprints:C-EUC0402
- added C65, C66, C67: CAP CER 0.1uF X7R 0402, rcl-modified-footprints:C-EUC0402
- R11, R12, R13, R3, R4, R5, R6, R8, R9: device rcl-modified-footprints:R-EU_R0603 -> rcl-modified-footprints:R-EU_R0402
- X1: value OUT0_P -> OUT2_P
- X2: value OUT0_N -> OUT2_N
- X3: value OUT2_P -> OUT0_P
- X6: value V_INPUT -> V_IN_EXT
Connections:
- removed net N$1: R6.2, R8.2, R9.2
- removed net NC_OUT2_N: IC1.OUT2_N
- removed net OUT0_N: IC1.OUT0_N, R4.2
- removed net OUT0_R_N: R12.2, R4.1, R8.1, X2.1
- new net NC_OUT0_N: IC1.OUT0_N
- new net OUT0_R_C_P: C64.2, R13.2, R9.1, X3.1
- new net OUT2_N: IC1.OUT2_N, R4.2
- new net OUT2_R_C_N: C52.2, R12.2, R8.1, X2.1
- new net OUT2_R_C_P: C50.2, R11.2, R6.1, X1.1
- new net OUT2_R_N: C52.1, R4.1
- net GND: now also C65.2, C66.2, C67.2
- net OUT0_P: now also R5.2; no longer R3.2
- net OUT0_R_P: now also C64.1, R5.1; no longer R11.2, R3.1, R6.1, X1.1
- net OUT2_P: now also R3.2; no longer R5.2
- net OUT2_R_P: now also C50.1, R3.1; no longer R13.2, R5.1, R9.1, X3.1
- net PP_P1V8_VDDO: now also C65.1, C66.1, C67.1, R6.2, R8.2, R9.2
Other:
- note added: "1.8V^2 / 50R = 64.8mW = 1/16W (so std. 0402 49.9R resistor can't be burnt out under any conditions)"
- note added: "CML output rise/fall times ~200ps Max stub ~ 1/3 * T(10-90) * c/n = 0.52" = 1.3cm"
- note added: "Optional VCM bias resistors"
- note removed: "Optional VCM refs"
- moved on the sheet: R11, R12, R13, R3, R4, R5, R6, R8, R9, X1, X2, X3
