File: meng-spad-quenching/active-quenching/aqc-rev4/aqc-rev4.sch (EAGLE design)
At the start: 285 parts, among them IC1 TPS7A4901, IC10 LT1534-1, IC11 HFA3134, IC12 HFA3134, IC13 HFA3134, IC14 LTC1711, IC15 NC7SV74K8X, IC16 74AHC1G14DCK, IC17 NL17SZ125, IC18 74AHC1G04DCK, IC19 74AHC1G32DCK, IC2 TPS7A4901, IC20 NC7WZ16P6X, IC21 74AHC1G08DCK, IC22 74AHC1G08DCK, IC23 HFA3134, IC24 TLV272DGK, IC25 THAT320, IC26 TLV272DGK, IC27 HFA3134, IC28 TLV271DBV, IC29 USBLC6-2SC6Y, IC3 LT1534-1, IC30 STM32F411RE, IC31 MAX5725, IC32 LM1117, IC4 ADCMP582, IC5 HFA3134, IC6 HFA3135, IC7 DS1100LU-45+, IC8 HFA3135, IC9 TPS7A3001, M1 BSS806N, M2 BSS806N, Q1 DMG2305UX-13, SW1 MCU_RST, T1 MMBTH10−4LT1G, U1 MCP4725, U2 SN65EPT22DGK, U3 SN65EPT21DGK, X1 CONN_PULLDN_SENSE, X2 CONN_FORCE_QUENCH, X3 KEYSTONE-7774, X4 CONN_SPAD, X5 CONN_PHOTON_COUNTER, X6 KEYSTONE-7774, X7 CONN_SMU, X8 61729-0010BLF

Commit message: Started aqc-rev4 design files by copying over aqc-rev3
Other:
- note removed: "f_sw = 100kHz"
