File: meng-spad-quenching/passive-quenching/pqc-rev3/pqc-rev3.brd (EAGLE design)
At the start: 38.1 x 25.4 mm, 62 parts, among them IC1 TPS7A4901, IC2 OPA858, IC3 OPA858, IC4 LM8261, Q1 NTR5105P, Q2 BSS123LT1G, Q3 NUD3160LT1G, X1 VIN_BIAS, X2 SPAD, X3 SIGNAL_OUT, X4 VIN_PWR

Commit message: Fixed filenames
Changed lines of the file:
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@@
 <contactref element="X2" pad="G@1"/>
 <polygon width="0.508" layer="16">
-<vertex x="-1" y="38.1"/>
-<vertex x="80.6825" y="38.1"/>
-<vertex x="81" y="-1"/>
+<vertex x="-1" y="30.48"/>
+<vertex x="40.64" y="30.48"/>
+<vertex x="40.64" y="0"/>
 <vertex x="-1" y="-1"/>
 </polygon>
@@
 <polygon width="0.254" layer="1" isolate="0.4064" rank="2">
 <vertex x="0" y="25.4"/>
-<vertex x="38.1" y="26.035"/>
-<vertex x="38.1" y="0.635"/>
+<vertex x="38.1" y="25.4"/>
+<vertex x="38.1" y="0"/>
 <vertex x="0" y="0"/>
 </polygon>

Commit message: work on BOMs
Parts:
- C12: value C_TUNE1 -> DNP
- C14: value C_TUNE2 -> DNP
- C17: value C_SNS -> CAP CER 10PF 250V C0G/NP0 0603
- C19: value C_FB2 -> DNP
- C20: value C_FB1 -> CAP CER 0.1PF 50V C0G/NP0 0402
- C3: value CAP CER 10000PF 25V X7R 0603 10% -> DNP
- D1: value DF2B36FU,H3F -> D55V0M1B2WS-7
- D3: value DF2B36FU,H3F -> DNP
- IC1: value TPS7A4901 -> TPS79850
- IC2: value OPA858 -> DNP
- R1: value RES SMD 76.8K OHM 1% 1/10W 0603 -> 0R JUMPER 0603
- R10: value R_FB2 -> RES SMD 100 OHM 1% 0402
- R11: value R_FB1 -> RES SMD 1K OHM 1% 0402
- R3: value RES SMD 24K OHM 1% 1/10W 0603 -> DNP
- R4: value R_TIA -> DNP
- R5: value R_Q -> RES SMD 100K OHM 1% 0805
- R6: value R_SNS1 -> DNP
- R7: value RES SMD 50 OHM 1% 0603 -> DNP
- R8: value R_SNS -> RES SMD 50 OHM 1% 0402
Connections:
- net LDO_P5V0_NR_SS_CH1 renamed LDO_P5V0_NR_SS

Commit message: Started aqc-rev4 design files by copying over aqc-rev3
Parts:
- C8: value CAP CER 10000PF 25V X7R 0603 10% -> CAP CER 10000PF 25V C0G 0603
- C9: value CAP CER 10NF 50V X7R 0603 -> CAP CER 10000PF 50V X7R 0603
Changed lines of the file:
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@@
 <attribute name="NAME" x="19.03375" y="23.16125" size="0.8128" layer="25" font="vector" ratio="16"/>
 </element>
-<element name="C8" library="rcl-modified-footprints" package="C0603" package3d_urn="urn:adsk.eagle:package:23616/2" value="CAP CER 10000PF 25V X7R 0603 10%" x="25.4" y="20.6375" smashed="yes">
+<element name="C8" library="rcl-modified-footprints" package="C0603" package3d_urn="urn:adsk.eagle:package:23616/2" value="CAP CER 10000PF 25V C0G 0603" x="25.4" y="20.6375" smashed="yes">
 <attribute name="NAME" x="24.4475" y="22.70125" size="0.8128" layer="25" font="vector" ratio="16"/>
 </element>
@@
 <attribute name="TP_SIGNAL_NAME" value="" x="18.415" y="5.23875" size="1" layer="37"/>
 </element>
-<element name="C9" library="rcl-modified-footprints" package="C0603" package3d_urn="urn:adsk.eagle:package:23616/2" value="CAP CER 10NF 50V X7R 0603" x="9.36625" y="18.335625" smashed="yes">
+<element name="C9" library="rcl-modified-footprints" package="C0603" package3d_urn="urn:adsk.eagle:package:23616/2" value="CAP CER 10000PF 50V X7R 0603" x="9.36625" y="18.335625" smashed="yes">
 <attribute name="NAME" x="10.795" y="18.494375" size="0.8128" layer="25" font="vector" ratio="16"/>
 </element>

Commit message: misc sync
Parts:
- IC2: value DNP -> OPA858
Changed lines of the file:
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@@
 <attribute name="NAME" x="15.24" y="17.30375" size="0.8128" layer="25" font="vector" ratio="16" rot="R90"/>
 </element>
-<element name="IC2" library="meng" package="WSON8" value="DNP" x="19.05" y="15.875" smashed="yes">
+<element name="IC2" library="meng" package="WSON8" value="OPA858" x="19.05" y="15.875" smashed="yes">
 <attribute name="NAME" x="20.6375" y="15.39875" size="0.8128" layer="25" font="vector" ratio="16"/>
 <attribute name="VALUE" x="20.6375" y="16.35125" size="0.8128" layer="27" font="vector" ratio="16"/>
