File: isg-pico-filter-breakout-rev1/isg-pico-filter-breakout-rev1.brd (EAGLE design)
At the start: 66 x 91.4 mm, 80 parts, among them IC1 PICO_BAREDIE, U1 OPA2380AIDGKT, U2 OPA2380AIDGKT, U3 OPA2380AIDGKT, U4 OPA2380AIDGKT, U5 OPA2380AIDGKT

Commit message: TVS diodes
Parts:
- C10, C11, C13, C14, C7, C8: value CAP CER 1PF C0G 0603 -> CAP CER 0.1UF X7R 0603
- C16, C17, C18, C19, C20, C3: value CAP CER 0.1UF X7R 0603 -> CAP CER 1PF C0G 0603
- H1, H2: value MOUNT-PAD-ROUND3.2 -> MOUNT-PAD-1/4-20-OPTICAL; device holes:3,2-PAD -> isg-custom:MOUNT-PAD-1/4-20
- H5, H6: value MOUNT-PAD-1/4-20-OPTICAL -> MOUNT-PAD-ROUND3.2; device isg-custom:MOUNT-PAD-1/4-20 -> holes:3,2-PAD
- R1, R2, R3, R4, R5: value RES SMD 1M OHM 1% 0603 -> RES SMD 49.9 OHM 1% 0603
- R16, R18, R20: value RES SMD 4.7K OHM 1% 0603 -> RES SMD 49.9 OHM 1% 0603
- R21, R23, R25: value RES SMD 49.9 OHM 1% 0603 -> RES SMD 4.7K OHM 1% 0603
- R26, R27, R28, R29, R30: value RES SMD 49.9 OHM 1% 0603 -> RES SMD 1M OHM 1% 0603
- moved H7 91.6 mm to (7.62, 7.62)
- moved H8 91.6 mm to (58.4, 7.62)
- moved H1 82.1 mm to (7.62, 83.8)
- moved H2 82.1 mm to (58.4, 83.8)
- moved H3 35.6 mm to (15.2, 77.5)
- moved H4 35.6 mm to (50.8, 77.5)
- moved C21 26.5 mm to (19.1, 53.3), turned to 180 degrees
- moved C11 24.6 mm to (16.2, 61.9), turned to 270 degrees
- moved R22 21.9 mm to (36.2, 58.1), turned to 90 degrees
- moved R24 21.9 mm to (43.2, 58.1), turned to 90 degrees
- moved C5 21.0 mm to (47.0, 67.9)
- moved R17 21.0 mm to (16.8, 58.1)
- moved R19 21.0 mm to (23.8, 58.1)
- moved R26 20.2 mm to (19.1, 57.1), turned to 180 degrees
- moved R5 20.2 mm to (47.0, 71.8)
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- renumbered D1 to D109, D10 to D101, D11 to D100, D2 to D108, D3 to D110, D4 to D107, D5 to D106, D6 to D105, D7 to D104, D8 to D103, D9 to D102, JP1 to JP100, JP2 to JP103, JP3 to JP102, JP4 to JP101
Connections:
- net +5V: now also C10.1, C7.1, C8.1; no longer C12.1, C15.1, C3.1
- net -5V: now also C11.2, C12.2, C13.2, C14.2, C15.2, R21.2, R23.2, R25.2; no longer C17.2, C18.2, C19.2, C20.2, C21.2, R16.2, R18.2, R20.2
- net F1_PD1_K: now also C16.1, R26.1; no longer C1.1, R1.1
- net F1_PD1_VOUT: now also C16.2, R16.1, R17.1, R26.2; no longer C1.2, R1.2, R11.1, R21.1
- net F1_PD1_VOUT_R: now also R16.2; no longer R21.2
- net F2_PD1_K: now also C17.1, R27.1; no longer C4.1, R3.1
- net F2_PD1_VOUT: now also C17.2, R18.1, R19.1, R27.2; no longer C4.2, R13.1, R23.1, R3.2
- net F2_PD1_VOUT_R: now also R18.2; no longer R23.2
- net F2_PD2_K: now also C1.1, R6.1; no longer C2.1, R2.1
- net F2_PD2_VOUT: now also C1.2, R1.1, R11.1, R6.2; no longer C2.2, R12.1, R2.2, R22.1
- net F2_PD2_VOUT_R: now also R1.2; no longer R22.2
- net F3_PD1_K: now also C3.1, R8.1; no longer C8.1, R6.1
- net F3_PD1_VOUT: now also C3.2, R13.1, R3.1, R8.2; no longer C8.2, R16.1, R26.1, R6.2
- net F3_PD1_VOUT_R: now also R3.2; no longer R26.2
- net F3_PD2_K: now also C18.1, R28.1; no longer C7.1, R5.1
- net F3_PD2_VOUT: now also C18.2, R20.1, R21.1, R28.2; no longer C7.2, R15.1, R25.1, R5.2
- net F3_PD2_VOUT_R: now also R20.2; no longer R25.2
- net F3_PD3_K: now also C2.1, R7.1; no longer C5.1, R4.1
- net F3_PD3_VOUT: now also C2.2, R12.1, R2.1, R7.2; no longer C5.2, R14.1, R24.1, R4.2
- net F3_PD3_VOUT_R: now also R2.2; no longer R24.2
- net F4_PD1_K: now also C5.1; no longer C14.1
- net F4_PD1_VOUT: now also C5.2, R15.1, R5.1; no longer C14.2, R20.1, R30.1
- net F4_PD1_VOUT_R: now also R5.2; no longer R30.2
- net F4_PD2_K: now also C20.1, R30.1; no longer C13.1, R9.1
- net F4_PD2_VOUT: now also C20.2, R24.1, R25.1, R30.2; no longer C13.2, R19.1, R29.1, R9.2
- net F4_PD2_VOUT_R: now also R24.2; no longer R29.2
- net F4_PD3_K: now also C4.1, R9.1; no longer C11.1, R8.1
- net F4_PD3_VOUT: now also C4.2, R14.1, R4.1, R9.2; no longer C11.2, R18.1, R28.1, R8.2
- net F4_PD3_VOUT_R: now also R4.2; no longer R28.2
- net F4_PD4_K: now also C19.1, R29.1; no longer C10.1, R7.1
- net F4_PD4_VOUT: now also C19.2, R22.1, R23.1, R29.2; no longer C10.2, R17.1, R27.1, R7.2
- net F4_PD4_VOUT_R: now also R22.2; no longer R27.2
- net GND: now also C10.2, C11.1, C12.1, C13.1, C14.1, C15.1, C21.2, C7.2, C8.2, H1.MOUNT, H2.MOUNT, H5.B3,2, H6.B3,2; no longer C12.2, C15.2, C16.2, C17.1, C18.1, C19.1, C20.1, C21.1, C3.2, H1.B3,2, H2.B3,2, H5.MOUNT, H6.MOUNT
- net PD_BIAS_N: now also C21.1; no longer C16.1
Other:
- board text added: "isg-pico-filter-breakout-rev1 kramnik@berkeley.edu vlada@berkeley.edu"
