File: isg-pico-filter-breakout-rev1/isg-pico-filter-breakout-rev1.sch (EAGLE design)
At the start: 51 parts, among them IC1 PICO_BAREDIE, U1 OPA2380AIDGKT, U2 OPA2380AIDGKT, U3 OPA2380AIDGKT, U4 OPA2380AIDGKT, U5 OPA2380AIDGKT, X3 PD_BIAS_N

Commit message: work on TIA layout
Parts:
- removed X3: PD_BIAS_N, con-coax:SMA-142-0701-881/886
- added JP1: (no value), pinhead:PINHD-2X10
- added JP2: TIA_OUT, pinhead:PINHD-2X10
- added R21, R22, R23, R24, R25, R26, R27, R28, R29, R30: RES SMD 49.9 OHM 1% 0603, rcl-modified-footprints:R-EU_R0603
- added X1, X2: 1365-20, con-leotronics:1365-20
Connections:
- new net +5V: C12.1, C15.1, C3.1, C6.1, C9.1, JP1.19, U1.V+, U2.V+, U3.V+, U4.V+, U5.V+
- new net -5V: JP1.1, R11.2, R12.2, R13.2, R14.2, R15.2, R16.2, R17.2, R18.2, R19.2, R20.2
- new net N$1: IC1.F1_H1_A, JP1.20
- new net N$10: IC1.F4_H1_A, JP1.2
- new net N$11: C4.2, R13.1, R23.1, R3.2, U2.OUT_A
- new net N$12: JP2.19, R21.2
- new net N$13: JP2.17, R22.2
- new net N$14: JP2.15, R23.2
- new net N$15: JP2.13, R24.2
- new net N$16: JP2.11, R25.2
- new net N$17: JP2.9, R26.2
- new net N$18: JP2.7, R27.2
- new net N$19: JP2.5, R28.2
- new net N$20: JP2.3, R29.2
- new net N$21: JP2.1, R30.2
- new net N$8: IC1.F4_H3_A, JP1.6
- new net N$9: IC1.F4_H2_A, JP1.4
- net F1_PD1_VOUT: now also R21.1
- net F2_PD1_VOUT: now also R22.1; no longer C4.2, R13.1, R3.2, U2.OUT_A
- net F3_PD1_VOUT: now also R26.1
- net F3_PD2_VOUT: now also R25.1
- net F3_PD3_VOUT: now also R24.1
- net F4_PD1_VOUT: now also R30.1
- net F4_PD2_VOUT: now also R29.1
- net F4_PD3_VOUT: now also R28.1
- net F4_PD4_VOUT: now also R27.1
- net GND: now also IC1.F1_H1_B, IC1.F2_H1_B, IC1.F2_H2_B, IC1.F3_H1_B, IC1.F3_H2_B, IC1.F3_H3_B, IC1.F4_H1_B, IC1.F4_H2_B, IC1.F4_H3_B, IC1.F4_H4_B, JP1.11, JP1.13, JP1.15, JP1.17, JP1.3, JP1.5, JP1.7, JP1.9, JP2.10, JP2.12, JP2.14, JP2.16, JP2.18, JP2.2, JP2.20, JP2.4, JP2.6, JP2.8; no longer X3.2
- net N$2: now also IC1.F2_H2_A, JP1.18; no longer R11.2, R12.2
- net N$3: now also IC1.F2_H1_A, JP1.16; no longer R13.2, R14.2
- net N$4: now also IC1.F3_H3_A, JP1.14; no longer R15.2, R16.2
- net N$5: now also IC1.F3_H2_A, JP1.12; no longer R17.2, R18.2
- net N$6: now also IC1.F3_H1_A, JP1.10; no longer C12.1, C15.1, C3.1, C6.1, C9.1, U1.V+, U2.V+, U3.V+, U4.V+, U5.V+
- net N$7: now also IC1.F4_H4_A, JP1.8; no longer R19.2, R20.2
- net PD_BIAS_N: no longer X3.1
Other:
- note added: "OPA380 can drive up to 500pF pure cap load, add resistors for damping"

Commit message: TIAs routed to 0.1" header
Connections:
- net N$12 renamed F1_PD1_VOUT_R
- net N$13 renamed F2_PD2_VOUT_R
- net N$14 renamed F2_PD1_VOUT_R
- net N$15 renamed F3_PD3_VOUT_R
- net N$16 renamed F3_PD2_VOUT_R
- net N$17 renamed F3_PD1_VOUT_R
- net N$18 renamed F4_PD4_VOUT_R
- net N$19 renamed F4_PD3_VOUT_R
- net N$20 renamed F4_PD2_VOUT_R
- net N$21 renamed F4_PD1_VOUT_R
- removed net N$11: C4.2, R13.1, R23.1, R3.2, U2.OUT_A
- new net F2_PD2_VOUT: C2.2, R12.1, R2.2, R22.1, U1.OUT_B
- net +5V: now also JP2.20; no longer JP1.19
- net -5V: now also JP2.2; no longer JP1.1
- net F2_PD1_VOUT: now also C4.2, R13.1, R23.1, R3.2, U2.OUT_A; no longer C2.2, R12.1, R2.2, R22.1, U1.OUT_B
- net GND: no longer JP2.2, JP2.20
Other:
- moved on the sheet: JP2

Commit message: first-pass routing done
Parts:
- removed X1, X2: 1365-20, con-leotronics:1365-20
- added C17, C18, C19, C20, C21: CAP CER 0.1UF X7R 0603, rcl-modified-footprints:C-EUC0603
- added JP3, JP4: HEATERS, isg-custom:FFSD-08-D-12.00-01-N
- C12, C15, C16, C3, C6, C9: value CAP CER 100NF X7R 0603 -> CAP CER 0.1UF X7R 0603
- JP1: value (none) -> HEATERS
Connections:
- removed net N$1: IC1.F1_H1_A, JP1.20
- removed net N$10: IC1.F4_H1_A, JP1.2
- removed net N$2: IC1.F2_H2_A, JP1.18
- removed net N$3: IC1.F2_H1_A, JP1.16
- removed net N$4: IC1.F3_H3_A, JP1.14
- removed net N$5: IC1.F3_H2_A, JP1.12
- removed net N$6: IC1.F3_H1_A, JP1.10
- removed net N$7: IC1.F4_H4_A, JP1.8
- removed net N$8: IC1.F4_H3_A, JP1.6
- removed net N$9: IC1.F4_H2_A, JP1.4
- new net F1_H1_A: IC1.F1_H1_A, JP1.20, JP4.20
- new net F2_H1_A: IC1.F2_H1_A, JP1.16, JP4.16
- new net F2_H2_A: IC1.F2_H2_A, JP1.18, JP4.18
- new net F3_H1_A: IC1.F3_H1_A, JP1.10, JP4.10
- new net F3_H2_A: IC1.F3_H2_A, JP1.12, JP4.12
- new net F3_H3_A: IC1.F3_H3_A, JP1.14, JP4.14
- new net F4_H1_A: IC1.F4_H1_A, JP1.2, JP4.2
- new net F4_H2_A: IC1.F4_H2_A, JP1.4, JP4.4
- new net F4_H3_A: IC1.F4_H3_A, JP1.6, JP4.6
- new net F4_H4_A: IC1.F4_H4_A, JP1.8, JP4.8
- net +5V: now also JP3.1
- net -5V: now also C17.2, C18.2, C19.2, C20.2, C21.2, JP3.19
- net F1_PD1_VOUT_R: now also JP3.2
- net F2_PD1_VOUT_R: now also JP3.6
- net F2_PD2_VOUT_R: now also JP3.4
- net F3_PD1_VOUT_R: now also JP3.12
- net F3_PD2_VOUT_R: now also JP3.10
- net F3_PD3_VOUT_R: now also JP3.8
- net F4_PD1_VOUT_R: now also JP3.20
- net F4_PD2_VOUT_R: now also JP3.18
- net F4_PD3_VOUT_R: now also JP3.16
- net F4_PD4_VOUT_R: now also JP3.14
- net GND: now also C17.1, C18.1, C19.1, C20.1, C21.1, JP1.1, JP1.19, JP3.11, JP3.13, JP3.15, JP3.3, JP3.5, JP3.7, JP3.9, JP4.1, JP4.11, JP4.13, JP4.15, JP4.17, JP4.19, JP4.3, JP4.5, JP4.7, JP4.9; no longer JP2.4
- net PD_BIAS_N: now also JP2.4, JP3.17
Other:
- note added: "FFSD-08-D-12.00-01-N"

Commit message: Added ESD diodes
Parts:
- added D1, D10, D11, D2, D3, D4, D5, D6, D7, D8, D9: DF2B36FU,H3F, diode:DIODE-SOD323-W
Connections:
- net F1_H1_A: now also D1.C
- net F2_H1_A: now also D4.C
- net F2_H2_A: now also D2.C
- net F3_H1_A: now also D7.C
- net F3_H2_A: now also D6.C
- net F3_H3_A: now also D5.C
- net F4_H1_A: now also D11.C
- net F4_H2_A: now also D10.C
- net F4_H3_A: now also D9.C
- net F4_H4_A: now also D8.C
- net GND: now also D1.A, D10.A, D11.A, D2.A, D3.C, D4.A, D5.A, D6.A, D7.A, D8.A, D9.A
- net PD_BIAS_N: now also D3.A
Other:
- note added: "28V ESD"
- moved on the sheet: JP3

Commit message: TVS diodes
Parts:
- C10, C11, C13, C14, C7, C8: value CAP CER 1PF C0G 0603 -> CAP CER 0.1UF X7R 0603
- C16, C17, C18, C19, C20, C3: value CAP CER 0.1UF X7R 0603 -> CAP CER 1PF C0G 0603
- H1, H2: value MOUNT-PAD-ROUND3.2 -> MOUNT-PAD-1/4-20-OPTICAL; device holes:MOUNT-PAD-ROUND3.2 -> isg-custom:MOUNT-PAD-1/4-20-OPTICAL
- H5, H6: value MOUNT-PAD-1/4-20-OPTICAL -> MOUNT-PAD-ROUND3.2; device isg-custom:MOUNT-PAD-1/4-20-OPTICAL -> holes:MOUNT-PAD-ROUND3.2
- R1, R2, R3, R4, R5: value RES SMD 1M OHM 1% 0603 -> RES SMD 49.9 OHM 1% 0603
- R16, R18, R20: value RES SMD 4.7K OHM 1% 0603 -> RES SMD 49.9 OHM 1% 0603
- R21, R23, R25: value RES SMD 49.9 OHM 1% 0603 -> RES SMD 4.7K OHM 1% 0603
- R26, R27, R28, R29, R30: value RES SMD 49.9 OHM 1% 0603 -> RES SMD 1M OHM 1% 0603
- renumbered D1 to D109, D10 to D101, D11 to D100, D2 to D108, D3 to D110, D4 to D107, D5 to D106, D6 to D105, D7 to D104, D8 to D103, D9 to D102, JP1 to JP100, JP2 to JP103, JP3 to JP102, JP4 to JP101
Connections:
- net +5V: now also C10.1, C7.1, C8.1; no longer C12.1, C15.1, C3.1
- net -5V: now also C11.2, C12.2, C13.2, C14.2, C15.2, R21.2, R23.2, R25.2; no longer C17.2, C18.2, C19.2, C20.2, C21.2, R16.2, R18.2, R20.2
- net F1_PD1_K: now also C16.1, R26.1; no longer C1.1, R1.1
- net F1_PD1_VOUT: now also C16.2, R16.1, R17.1, R26.2; no longer C1.2, R1.2, R11.1, R21.1
- net F1_PD1_VOUT_R: now also R16.2; no longer R21.2
- net F2_PD1_K: now also C17.1, R27.1; no longer C4.1, R3.1
- net F2_PD1_VOUT: now also C17.2, R18.1, R19.1, R27.2; no longer C4.2, R13.1, R23.1, R3.2
- net F2_PD1_VOUT_R: now also R18.2; no longer R23.2
- net F2_PD2_K: now also C1.1, R6.1; no longer C2.1, R2.1
- net F2_PD2_VOUT: now also C1.2, R1.1, R11.1, R6.2; no longer C2.2, R12.1, R2.2, R22.1
- net F2_PD2_VOUT_R: now also R1.2; no longer R22.2
- net F3_PD1_K: now also C3.1, R8.1; no longer C8.1, R6.1
- net F3_PD1_VOUT: now also C3.2, R13.1, R3.1, R8.2; no longer C8.2, R16.1, R26.1, R6.2
- net F3_PD1_VOUT_R: now also R3.2; no longer R26.2
- net F3_PD2_K: now also C18.1, R28.1; no longer C7.1, R5.1
- net F3_PD2_VOUT: now also C18.2, R20.1, R21.1, R28.2; no longer C7.2, R15.1, R25.1, R5.2
- net F3_PD2_VOUT_R: now also R20.2; no longer R25.2
- net F3_PD3_K: now also C2.1, R7.1; no longer C5.1, R4.1
- net F3_PD3_VOUT: now also C2.2, R12.1, R2.1, R7.2; no longer C5.2, R14.1, R24.1, R4.2
- net F3_PD3_VOUT_R: now also R2.2; no longer R24.2
- net F4_PD1_K: now also C5.1; no longer C14.1
- net F4_PD1_VOUT: now also C5.2, R15.1, R5.1; no longer C14.2, R20.1, R30.1
- net F4_PD1_VOUT_R: now also R5.2; no longer R30.2
- net F4_PD2_K: now also C20.1, R30.1; no longer C13.1, R9.1
- net F4_PD2_VOUT: now also C20.2, R24.1, R25.1, R30.2; no longer C13.2, R19.1, R29.1, R9.2
- net F4_PD2_VOUT_R: now also R24.2; no longer R29.2
- net F4_PD3_K: now also C4.1, R9.1; no longer C11.1, R8.1
- net F4_PD3_VOUT: now also C4.2, R14.1, R4.1, R9.2; no longer C11.2, R18.1, R28.1, R8.2
- net F4_PD3_VOUT_R: now also R4.2; no longer R28.2
- net F4_PD4_K: now also C19.1, R29.1; no longer C10.1, R7.1
- net F4_PD4_VOUT: now also C19.2, R22.1, R23.1, R29.2; no longer C10.2, R17.1, R27.1, R7.2
- net F4_PD4_VOUT_R: now also R22.2; no longer R27.2
- net GND: now also C10.2, C11.1, C12.1, C13.1, C14.1, C15.1, C21.2, C7.2, C8.2; no longer C12.2, C15.2, C16.2, C17.1, C18.1, C19.1, C20.1, C21.1, C3.2
- net PD_BIAS_N: now also C21.1; no longer C16.1
Other:
- moved on the sheet: C1, C10, C11, C12, C13, C14, C15, C16, C17, C18, C19, C2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
